Commit message: start merge ros2 controllers gazebo and moveit

File: robot_description/urdf/moveit_ros2_control.xacro (robot description, xacro)
@@ -1,10 +1,9 @@
 <?xml version="1.0"?>
-<robot xmlns:xacro="http://www.ros.org/wiki/xacro">
-    <xacro:macro name="crx10ial_ros2_control" params="name initial_positions_file">
+<robot name="crx10ial" xmlns:xacro="http://www.ros.org/wiki/xacro">
+    <xacro:macro name="ros2_control" params="name initial_positions_file">
         <xacro:property name="initial_positions" value="${load_yaml(initial_positions_file)['initial_positions']}"/>
         <!-- This is the controller that is only used when MoveIt is launched without also launching Gazebo -->
         <ros2_control name="${name}" type="system">
             <hardware>
-                <!-- By default, set up controllers for simulation. This won't work on real hardware -->
                 <plugin>mock_components/GenericSystem</plugin>
             </hardware>

File: robot_description/urdf/robot.xacro (robot description, xacro)
@@ -7,4 +7,5 @@
   <!-- Gazebo Controllers -->
   <xacro:include filename="$(find robot_description)/urdf/simulation_interface.xacro"/>
+  <xacro:ros2_control name="GazeboSystem" initial_positions_file="$(find robot_moveit_config)/config/initial_positions.yaml"/>
   <xacro:crx10ial/>
 </robot>

File: robot_description/urdf/robot_moveit.xacro (robot description, xacro)
@@ -7,5 +7,5 @@
   <!-- MoveIt controllers -->
   <xacro:include filename="$(find robot_description)/urdf/moveit_ros2_control.xacro" />
-  <xacro:crx10ial_ros2_control name="FakeSystem" initial_positions_file="$(find robot_moveit_config)/config/initial_positions.yaml"/>
+  <xacro:ros2_control name="FakeSystem" initial_positions_file="$(find robot_moveit_config)/config/initial_positions.yaml"/>
   <xacro:crx10ial/>
 </robot>

File: robot_description/urdf/simulation_interface.xacro (robot description, xacro)
@@ -1,103 +1,106 @@
 <?xml version="1.0"?>
 <robot name="crx10ial" xmlns:xacro="http://www.ros.org/wiki/xacro">
-    <!-- Simulation ros2_control interface -->
-    <ros2_control name="GazeboSystem" type="system">
-        <hardware>
-            <plugin>gazebo_ros2_control/GazeboSystem</plugin>
-        </hardware>
-        <joint name="J1">
-            <command_interface name="position">
-                <param name="min">{-2*pi}</param>
-                <param name="max">{2*pi}</param>
-            </command_interface>
-            <state_interface name="position">
-            <param name="initial_value">0</param>
-            </state_interface>
-            <state_interface name="velocity"/>
-            <state_interface name="effort"/>
-        </joint>
-        <joint name="J2">
-            <command_interface name="position">
-                <param name="min">{-2*pi}</param>
-                <param name="max">{2*pi}</param>
-            </command_interface>
-            <state_interface name="position">
-            <param name="initial_value">0</param>
-            </state_interface>
-            <state_interface name="velocity"/>
-            <state_interface name="effort"/>
-        </joint>
-        <joint name="J3">
-            <command_interface name="position">
-                <param name="min">{-1* pi}</param>
-                <param name="max">{pi}</param>
-            </command_interface>
-            <state_interface name="position">
-            <param name="initial_value">0</param>
-            </state_interface>
-            <state_interface name="velocity"/>
-            <state_interface name="effort"/>
-        </joint>
-        <joint name="J4">
-            <command_interface name="position">
-                <param name="min">{-2*pi}</param>
-                <param name="max">{2*pi}</param>
-            </command_interface>
-            <state_interface name="position">
-            <param name="initial_value">0</param>
-            </state_interface>
-            <state_interface name="velocity"/>
-            <state_interface name="effort"/>
-        </joint>
-        <joint name="J5">
-            <command_interface name="position">
-                <param name="min">{-2*pi}</param>
-                <param name="max">{2*pi}</param>
-            </command_interface>
-            <state_interface name="position">
-            <param name="initial_value">0</param>
-            </state_interface>
-            <state_interface name="velocity"/>
-            <state_interface name="effort"/>
-        </joint>
-        <joint name="J6">
-            <command_interface name="position">
-                <param name="min">{-2*pi}</param>
-                <param name="max">{2*pi}</param>
-            </command_interface>
-            <state_interface name="position">
-            <param name="initial_value">0</param>
-            </state_interface>
-            <state_interface name="velocity"/>
-            <state_interface name="effort"/>
-        </joint>
-    </ros2_control>
-    <!-- Gazebo plugins -->
-    <gazebo>
-        <plugin filename="libgazebo_ros2_control.so" name="gazebo_ros2_control">
-            <parameters>$(find robot_moveit_config)/config/ros2_controllers.yaml</parameters>
-        </plugin>
-    </gazebo>
-    <!-- Add colours to the robot in Gazebo -->
-    <gazebo reference="base_link">
-        <material>Gazebo/Black</material>
-    </gazebo>
-    <gazebo reference="J1_link">
-        <material>Gazebo/White</material>
-    </gazebo>
-    <gazebo reference="J2_link">
-        <material>Gazebo/White</material>
-    </gazebo>
-    <gazebo reference="J3_link">
-        <material>Gazebo/White</material>
-    </gazebo>
-    <gazebo reference="J4_link">
-        <material>Gazebo/White</material>
-    </gazebo>
-    <gazebo reference="J5_link">
-        <material>Gazebo/White</material>
-    </gazebo>
-    <gazebo reference="J6_link">
-        <material>Gazebo/Black</material>
-    </gazebo>
+    <xacro:macro name="ros2_control" params="name initial_positions_file moveit_only:=false">
+        <xacro:property name="initial_positions" value="${load_yaml(initial_positions_file)['initial_positions']}"/>
+        <!-- Simulation ros2_control interface -->
+        <ros2_control name="${name}" type="system">
+            <hardware>
+                <plugin>gazebo_ros2_control/GazeboSystem</plugin>
+            </hardware>
+            <joint name="J1">
+                <command_interface name="position">
+                    <param name="min">{-2*pi}</param>
+                    <param name="max">{2*pi}</param>
+                </command_interface>
+                <state_interface name="position">
+                <param name="initial_value">${initial_positions['J1']}</param>
+                </state_interface>
+                <state_interface name="velocity"/>
+                <state_interface name="effort"/>
+            </joint>
+            <joint name="J2">
+                <command_interface name="position">
+                    <param name="min">{-2*pi}</param>
+                    <param name="max">{2*pi}</param>
+                </command_interface>
+                <state_interface name="position">
+                <param name="initial_value">${initial_positions['J2']}</param>
+                </state_interface>
+                <state_interface name="velocity"/>
+                <state_interface name="effort"/>
+            </joint>
+            <joint name="J3">
+                <command_interface name="position">
+                    <param name="min">{-1* pi}</param>
+                    <param name="max">{pi}</param>
+                </command_interface>
+                <state_interface name="position">
+                <param name="initial_value">${initial_positions['J3']}</param>
+                </state_interface>
+                <state_interface name="velocity"/>
+                <state_interface name="effort"/>
+            </joint>
+            <joint name="J4">
+                <command_interface name="position">
+                    <param name="min">{-2*pi}</param>
+                    <param name="max">{2*pi}</param>
+                </command_interface>
+                <state_interface name="position">
+                <param name="initial_value">${initial_positions['J4']}</param>
+                </state_interface>
+                <state_interface name="velocity"/>
+                <state_interface name="effort"/>
+            </joint>
+            <joint name="J5">
+                <command_interface name="position">
+                    <param name="min">{-2*pi}</param>
+                    <param name="max">{2*pi}</param>
+                </command_interface>
+                <state_interface name="position">
+                <param name="initial_value">${initial_positions['J5']}</param>
+                </state_interface>
+                <state_interface name="velocity"/>
+                <state_interface name="effort"/>
+            </joint>
+            <joint name="J6">
+                <command_interface name="position">
+                    <param name="min">{-2*pi}</param>
+                    <param name="max">{2*pi}</param>
+                </command_interface>
+                <state_interface name="position">
+                <param name="initial_value">${initial_positions['J6']}</param>
+                </state_interface>
+                <state_interface name="velocity"/>
+                <state_interface name="effort"/>
+            </joint>
+        </ros2_control>
+        <!-- Gazebo plugins -->
+        <gazebo>
+            <plugin filename="libgazebo_ros2_control.so" name="gazebo_ros2_control">
+                <parameters>$(find robot_moveit_config)/config/ros2_controllers.yaml</parameters>
+            </plugin>
+        </gazebo>
+        <!-- Add colours to the robot in Gazebo -->
+        <gazebo reference="base_link">
+            <material>Gazebo/Black</material>
+        </gazebo>
+        <gazebo reference="J1_link">
+            <material>Gazebo/White</material>
+        </gazebo>
+        <gazebo reference="J2_link">
+            <material>Gazebo/White</material>
+        </gazebo>
+        <gazebo reference="J3_link">
+            <material>Gazebo/White</material>
+        </gazebo>
+        <gazebo reference="J4_link">
+            <material>Gazebo/White</material>
+        </gazebo>
+        <gazebo reference="J5_link">
+            <material>Gazebo/White</material>
+        </gazebo>
+        <gazebo reference="J6_link">
+            <material>Gazebo/Black</material>
+        </gazebo>
+    </xacro:macro>
 </robot>

Commit message: replaced depricated load.yaml

File: robot_description/urdf/moveit_ros2_control.xacro (robot description, xacro)
@@ -2,5 +2,5 @@
 <robot name="crx10ial" xmlns:xacro="http://www.ros.org/wiki/xacro">
     <xacro:macro name="ros2_control" params="name initial_positions_file">
-        <xacro:property name="initial_positions" value="${load_yaml(initial_positions_file)['initial_positions']}"/>
+        <xacro:property name="initial_positions" value="${xacro.load_yaml(initial_positions_file)['initial_positions']}"/>
         <!-- This is the controller that is only used when MoveIt is launched without also launching Gazebo -->
         <ros2_control name="${name}" type="system">

File: robot_description/urdf/simulation_interface.xacro (robot description, xacro)
@@ -2,5 +2,5 @@
 <robot name="crx10ial" xmlns:xacro="http://www.ros.org/wiki/xacro">
     <xacro:macro name="ros2_control" params="name initial_positions_file moveit_only:=false">
-        <xacro:property name="initial_positions" value="${load_yaml(initial_positions_file)['initial_positions']}"/>
+        <xacro:property name="initial_positions" value="${xacro.load_yaml(initial_positions_file)['initial_positions']}"/>
         <!-- Simulation ros2_control interface -->
         <ros2_control name="${name}" type="system">
