Commit message: moveit and gazebo working, not with same controllers

File: robot_description/urdf/simulation_interface.xacro (robot description, xacro)
@@ -30,5 +30,5 @@
         <joint name="J3">
             <command_interface name="position">
-                <param name="min">{pi}</param>
+                <param name="min">{-1* pi}</param>
                 <param name="max">{pi}</param>
             </command_interface>
@@ -75,5 +75,4 @@
     <!-- Gazebo plugins -->
     <gazebo>
-        <!-- ros2_control -->
         <plugin filename="libgazebo_ros2_control.so" name="gazebo_ros2_control">
             <parameters>$(find robot_moveit_config)/config/ros2_controllers.yaml</parameters>

File: robot_moveit_config/config/crx10ial.ros2_control.xacro (robot description, xacro)
@@ -1,82 +1,54 @@
 <?xml version="1.0"?>
-<robot name="crx10ial" xmlns:xacro="http://www.ros.org/wiki/xacro">
-    <!-- Simulation ros2_control interface -->
-    <ros2_control name="GazeboSystem" type="system">
-        <hardware>
-            <plugin>gazebo_ros2_control/GazeboSystem</plugin>
-        </hardware>
-        <joint name="J1">
-            <command_interface name="position">
-                <param name="min">{-2*pi}</param>
-                <param name="max">{2*pi}</param>
-            </command_interface>
-            <state_interface name="position">
-                <param name="initial_value">0</param>
-            </state_interface>
-            <state_interface name="velocity"/>
-            <state_interface name="effort"/>
-        </joint>
-        <joint name="J2">
-            <command_interface name="position">
-                <param name="min">{-2*pi}</param>
-                <param name="max">{2*pi}</param>
-            </command_interface>
-            <state_interface name="position">
-                <param name="initial_value">0</param>
-            </state_interface>
-            <state_interface name="velocity"/>
-            <state_interface name="effort"/>
-        </joint>
-        <joint name="J3">
-            <command_interface name="position">
-                <param name="min">{pi}</param>
-                <param name="max">{pi}</param>
-            </command_interface>
-            <state_interface name="position">
-                <param name="initial_value">0</param>
-            </state_interface>
-            <state_interface name="velocity"/>
-            <state_interface name="effort"/>
-        </joint>
-        <joint name="J4">
-            <command_interface name="position">
-                <param name="min">{-2*pi}</param>
-                <param name="max">{2*pi}</param>
-            </command_interface>
-            <state_interface name="position">
-                <param name="initial_value">0</param>
-            </state_interface>
-            <state_interface name="velocity"/>
-            <state_interface name="effort"/>
-        </joint>
-        <joint name="J5">
-            <command_interface name="position">
-                <param name="min">{-2*pi}</param>
-                <param name="max">{2*pi}</param>
-            </command_interface>
-            <state_interface name="position">
-                <param name="initial_value">0</param>
-            </state_interface>
-            <state_interface name="velocity"/>
-            <state_interface name="effort"/>
-        </joint>
-        <joint name="J6">
-            <command_interface name="position">
-                <param name="min">{-2*pi}</param>
-                <param name="max">{2*pi}</param>
-            </command_interface>
-            <state_interface name="position">
-                <param name="initial_value">0</param>
-            </state_interface>
-            <state_interface name="velocity"/>
-            <state_interface name="effort"/>
-        </joint>
-    </ros2_control>
-    <!-- Gazebo plugins -->
-    <gazebo>
-        <!-- ros2_control -->
-        <plugin filename="libgazebo_ros2_control.so" name="gazebo_ros2_control">
-            <parameters>$(find robot_moveit_config)/config/ros2_controllers.yaml</parameters>
-        </plugin>
-    </gazebo>
+<robot xmlns:xacro="http://www.ros.org/wiki/xacro">
+    <xacro:macro name="crx10ial_ros2_control" params="name initial_positions_file">
+        <xacro:property name="initial_positions" value="${load_yaml(initial_positions_file)['initial_positions']}"/>
+        <ros2_control name="${name}" type="system">
+            <hardware>
+                <!-- By default, set up controllers for simulation. This won't work on real hardware -->
+                <plugin>mock_components/GenericSystem</plugin>
+            </hardware>
+            <joint name="J1">
+                <command_interface name="position"/>
+                <state_interface name="position">
+                  <param name="initial_value">${initial_positions['J1']}</param>
+                </state_interface>
+                <state_interface name="velocity"/>
+            </joint>
+            <joint name="J2">
+                <command_interface name="position"/>
+                <state_interface name="position">
+                  <param name="initial_value">${initial_positions['J2']}</param>
+                </state_interface>
+                <state_interface name="velocity"/>
+            </joint>
+            <joint name="J3">
+                <command_interface name="position"/>
+                <state_interface name="position">
+                  <param name="initial_value">${initial_positions['J3']}</param>
+                </state_interface>
+                <state_interface name="velocity"/>
+            </joint>
+            <joint name="J4">
+                <command_interface name="position"/>
+                <state_interface name="position">
+                  <param name="initial_value">${initial_positions['J4']}</param>
+                </state_interface>
+                <state_interface name="velocity"/>
+            </joint>
+            <joint name="J5">
+                <command_interface name="position"/>
+                <state_interface name="position">
+                  <param name="initial_value">${initial_positions['J5']}</param>
+                </state_interface>
+                <state_interface name="velocity"/>
+            </joint>
+            <joint name="J6">
+                <command_interface name="position"/>
+                <state_interface name="position">
+                  <param name="initial_value">${initial_positions['J6']}</param>
+                </state_interface>
+                <state_interface name="velocity"/>
+            </joint>
+        </ros2_control>
+    </xacro:macro>
 </robot>

File: robot_moveit_config/config/crx10ial.urdf.xacro (robot description, xacro)
@@ -1,8 +1,9 @@
 <?xml version="1.0"?>
 <robot xmlns:xacro="http://www.ros.org/wiki/xacro" name="crx10ial">
+    <xacro:arg name="initial_positions_file" default="initial_positions.yaml" />
     <!-- Import crx10ial urdf file -->
     <xacro:include filename="$(find robot_description)/urdf/robot.xacro" />
     <!-- Import control_xacro -->
-    <xacro:include filename="$(find robot_moveit_config)/config/crx10ial.ros2_control.xacro" />
-    <xacro:crx10ial/>
+    <xacro:include filename="crx10ial.ros2_control.xacro" />
+    <xacro:crx10ial_ros2_control name="FakeSystem" initial_positions_file="$(arg initial_positions_file)"/>
 </robot>

Commit message: Added Gazebo colours

File: robot_description/urdf/simulation_interface.xacro (robot description, xacro)
@@ -79,3 +79,25 @@
         </plugin>
     </gazebo>
+    <!-- Add colours to the robot in Gazebo -->
+    <gazebo reference="base_link">
+        <material>Gazebo/Black</material>
+    </gazebo>
+    <gazebo reference="J1_link">
+        <material>Gazebo/White</material>
+    </gazebo>
+    <gazebo reference="J2_link">
+        <material>Gazebo/White</material>
+    </gazebo>
+    <gazebo reference="J3_link">
+        <material>Gazebo/White</material>
+    </gazebo>
+    <gazebo reference="J4_link">
+        <material>Gazebo/White</material>
+    </gazebo>
+    <gazebo reference="J5_link">
+        <material>Gazebo/White</material>
+    </gazebo>
+    <gazebo reference="J6_link">
+        <material>Gazebo/Black</material>
+    </gazebo>
 </robot>

Commit message: small config and colour adjustments

File: robot_description/urdf/simulation_interface.xacro (robot description, xacro)
@@ -83,5 +83,5 @@
         <!-- Add colours to the robot in Gazebo -->
         <gazebo reference="base_link">
-            <material>Gazebo/Black</material>
+            <material>Gazebo/Road</material>
         </gazebo>
         <gazebo reference="J1_link">
@@ -101,5 +101,5 @@
         </gazebo>
         <gazebo reference="J6_link">
-            <material>Gazebo/Black</material>
+            <material>Gazebo/Road</material>
         </gazebo>
         <!-- Add colours to the end effector -->
