Commit message: combined the controllers

File: robot_description/urdf/robot.xacro (robot description, xacro)
@@ -1,14 +1,10 @@
 <?xml version="1.0"?>
 <robot name="crx10ial" xmlns:xacro="http://wiki.ros.org/xacro">
-  <!-- Arguments-->
-  <xacro:arg name="sim" default="false"/> <!-- Default left at false for MoveIt, needs fixing-->
   <!-- Utils -->
   <xacro:include filename="$(find robot_description)/urdf/utils.xacro" />
   <!-- Robot model-->
   <xacro:include filename="$(find robot_description)/urdf/robot.urdf.xacro"/>
-  <!-- Simulation interface-->
-  <xacro:if value="$(arg sim)">
-    <xacro:include filename = "$(find robot_description)/urdf/simulation_interface.xacro" />
-  </xacro:if>
+  <!-- Simulation interface, located in MoveIt package-->
+  <xacro:include filename = "$(find robot_description)/urdf/simulation_interface.xacro" />
   <xacro:crx10ial/>
 </robot>

File: robot_description/urdf/simulation_interface.xacro (robot description, xacro)
@@ -1,95 +1,100 @@
 <?xml version="1.0"?>
-<robot xmlns:xacro="http://ros.org/wiki/xacro">
-    <!-- Simulation ros2_control interface -->
-    <ros2_control name="IgnitionSystem" type="system">
-        <hardware>
-            <plugin>ign_ros2_control/IgnitionSystem</plugin>
-        </hardware>
-        <joint name="J1">
-            <command_interface name="position">
-                <param name="min">{-2*pi}</param>
-                <param name="max">{2*pi}</param>
-            </command_interface>
-            <state_interface name="position">
-                <param name="initial_value">0.0</param>
-            </state_interface>
-            <state_interface name="velocitiy"/>
-        </joint>
-        <joint name="J2">
-            <command_interface name="position">
-                <param name="min">{-2*pi}</param>
-                <param name="max">{2*pi}</param>
-            </command_interface>
-            <state_interface name="position">
-                <param name="initial_value">0.0</param>
-            </state_interface>
-            <state_interface name="velocitiy"/>
-        </joint>
-        <joint name="J3">
-            <command_interface name="position">
-                <param name="min">{pi}</param>
-                <param name="max">{pi}</param>
-            </command_interface>
-            <state_interface name="position">
-                <param name="initial_value">0.0</param>
-            </state_interface>
-            <state_interface name="velocitiy"/>
-        </joint>
-        <joint name="J4">
-            <command_interface name="position">
-                <param name="min">{-2*pi}</param>
-                <param name="max">{2*pi}</param>
-            </command_interface>
-            <state_interface name="position">
-                <param name="initial_value">0.0</param>
-            </state_interface>
-            <state_interface name="velocitiy"/>
-        </joint>
-        <joint name="J5">
-            <command_interface name="position">
-                <param name="min">{-2*pi}</param>
-                <param name="max">{2*pi}</param>
-            </command_interface>
-            <state_interface name="position">
-                <param name="initial_value">0.0</param>
-            </state_interface>
-            <state_interface name="velocitiy"/>
-        </joint>
-        <joint name="J6">
-            <command_interface name="position">
-                <param name="min">{-2*pi}</param>
-                <param name="max">{2*pi}</param>
-            </command_interface>
-            <state_interface name="position">
-                <param name="initial_value">0.0</param>
-            </state_interface>
-            <state_interface name="velocitiy"/>
-        </joint>
-    </ros2_control>
-    <!-- Gazebo plugins -->
-    <gazebo>
-        <!-- ros2_control -->
-        <plugin filename="ign_ros2_control-system" name="ign_ros2_control::IgnitionROS2ControlPlugin">
-            <parameters>$(find robot_moveit_config)/config/controller_params.yaml</parameters>
-        </plugin>
-        <plugin filename="libgazebo_ros2_control.so" name="gazebo_ros2_control">
-            <robotNamespace>/</robotNamespace>
-        </plugin>
-        <!-- IMU -->
-        <plugin filename="libignition-gazebo-imu-system.so" name="ignition::gazebo::systems::Imu"/>
-        <!-- Sensor plugins (nog van smart_diffbot)-->
-        <plugin filename="ignition-gazebo-sensors-system" name="ignition::gazebo::systems::Sensors">
-            <render_engine>ogre2</render_engine>
-        </plugin>
-    </gazebo>
-    <!-- Sensor simulation -->
-    <gazebo reference="imu_link">
-        <sensor name="imu" type="imu">
-            <always_on>1</always_on>
-            <update_rate>15</update_rate>
-            <visualize>false</visualize>
-            <topic>imu/data</topic>
-            <ignition_frame_id>imu_link</ignition_frame_id>
-        </sensor>
-    </gazebo>
+<robot xmlns:xacro="http://www.ros.org/wiki/xacro">
+    <xacro:macro name="crx10ial_ros2_control" params="name initial_positions_file">
+        <xacro:property name="initial_positions" value="${load_yaml(initial_positions_file)['initial_positions']}"/>
+        <!-- Simulation ros2_control interface -->
+        <ros2_control name="${name}" type="system">
+            <hardware>
+                <!-- By default, set up controllers for simulation. This won't work on real hardware -->
+                <plugin>mock_components/GenericSystem</plugin>
+                <plugin>ign_ros2_control/IgnitionSystem</plugin>
+            </hardware>
+            <joint name="J1">
+                <command_interface name="position">
+                    <param name="min">{-2*pi}</param>
+                    <param name="max">{2*pi}</param>
+                </command_interface>
+                <state_interface name="position">
+                  <param name="initial_value">${initial_positions['J1']}</param>
+                </state_interface>
+                <state_interface name="velocity"/>
+            </joint>
+            <joint name="J2">
+                <command_interface name="position">
+                    <param name="min">{-2*pi}</param>
+                    <param name="max">{2*pi}</param>
+                </command_interface>
+                <state_interface name="position">
+                  <param name="initial_value">${initial_positions['J2']}</param>
+                </state_interface>
+                <state_interface name="velocity"/>
+            </joint>
+            <joint name="J3">
+                <command_interface name="position">
+                    <param name="min">{pi}</param>
+                    <param name="max">{pi}</param>
+                </command_interface>
+                <state_interface name="position">
+                  <param name="initial_value">${initial_positions['J3']}</param>
+                </state_interface>
+                <state_interface name="velocity"/>
+            </joint>
+            <joint name="J4">
+                <command_interface name="position">
+                    <param name="min">{-2*pi}</param>
+                    <param name="max">{2*pi}</param>
+                </command_interface>
+                <state_interface name="position">
+                  <param name="initial_value">${initial_positions['J4']}</param>
+                </state_interface>
+                <state_interface name="velocity"/>
+            </joint>
+            <joint name="J5">
+                <command_interface name="position">
+                    <param name="min">{-2*pi}</param>
+                    <param name="max">{2*pi}</param>
+                </command_interface>
+                <state_interface name="position">
+                  <param name="initial_value">${initial_positions['J5']}</param>
+                </state_interface>
+                <state_interface name="velocity"/>
+            </joint>
+            <joint name="J6">
+                <command_interface name="position">
+                    <param name="min">{-2*pi}</param>
+                    <param name="max">{2*pi}</param>
+                </command_interface>
+                <state_interface name="position">
+                  <param name="initial_value">${initial_positions['J6']}</param>
+                </state_interface>
+                <state_interface name="velocity"/>
+            </joint>
+        </ros2_control>
+        <!-- Gazebo plugins -->
+        <gazebo>
+            <!-- ros2_control -->
+            <plugin filename="ign_ros2_control-system" name="ign_ros2_control::IgnitionROS2ControlPlugin">
+                <parameters>$(find robot_moveit_config)/config/controller_params.yaml</parameters>
+            </plugin>
+            <plugin filename="libgazebo_ros2_control.so" name="gazebo_ros2_control">
+                <robotNamespace>/</robotNamespace>
+            </plugin>
+            <!-- IMU -->
+            <plugin filename="libignition-gazebo-imu-system.so" name="ignition::gazebo::systems::Imu"/>
+            <!-- Sensor plugins (nog van smart_diffbot)-->
+            <plugin filename="ignition-gazebo-sensors-system" name="ignition::gazebo::systems::Sensors">
+                <render_engine>ogre2</render_engine>
+            </plugin>
+        </gazebo>
+        <!-- Sensor simulation -->
+        <gazebo reference="imu_link">
+            <sensor name="imu" type="imu">
+                <always_on>1</always_on>
+                <update_rate>15</update_rate>
+                <visualize>false</visualize>
+                <topic>imu/data</topic>
+                <ignition_frame_id>imu_link</ignition_frame_id>
+            </sensor>
+        </gazebo>
+    </xacro:macro>
 </robot>

File: robot_moveit_config/config/crx10ial.urdf.xacro (robot description, xacro)
@@ -4,6 +4,4 @@
     <!-- Import crx10ial urdf file -->
     <xacro:include filename="$(find robot_description)/urdf/robot.xacro" />
-    <!-- Import control_xacro -->
-    <xacro:include filename="crx10ial.ros2_control.xacro" />
-    <xacro:crx10ial_ros2_control name="FakeSystem" initial_positions_file="$(arg initial_positions_file)"/>
+    <xacro:crx10ial_ros2_control name="IgnitionSystem" initial_positions_file="$(arg initial_positions_file)"/>
 </robot>

Commit message: merged URDFs by using arguments

File: robot_description/urdf/robot.xacro (robot description, xacro)
@@ -3,4 +3,5 @@
   <!-- Arguments -->
   <xacro:arg name="moveit_only" default="false"/>
+  <xacro:arg name="gazebo_classic" default="false"/>
   <!-- Utils -->
   <xacro:include filename="$(find robot_description)/urdf/utils.xacro" />
@@ -10,5 +11,5 @@
   <xacro:unless value="$(arg moveit_only)">
     <xacro:include filename="$(find robot_description)/urdf/simulation_interface.xacro"/>
-    <xacro:ros2_control name="GazeboSystem" initial_positions_file="$(find robot_moveit_config)/config/initial_positions.yaml"/>
+    <xacro:ros2_control name="GazeboSystem" initial_positions_file="$(find robot_moveit_config)/config/initial_positions.yaml" gazebo_classic="$(arg gazebo_classic)"/>
   </xacro:unless>
   <!-- Load MoveIt Controllers if moveit_only is true -->

File: robot_description/urdf/simulation_interface.xacro (robot description, xacro)
@@ -1,10 +1,15 @@
 <?xml version="1.0"?>
 <robot name="crx10ial" xmlns:xacro="http://www.ros.org/wiki/xacro">
-    <xacro:macro name="ros2_control" params="name initial_positions_file moveit_only:=false">
+    <xacro:macro name="ros2_control" params="name initial_positions_file gazebo_classic">
         <xacro:property name="initial_positions" value="${xacro.load_yaml(initial_positions_file)['initial_positions']}"/>
         <!-- Simulation ros2_control interface -->
         <ros2_control name="${name}" type="system">
             <hardware>
-                <plugin>gazebo_ros2_control/GazeboSystem</plugin>
+                <xacro:if value="${gazebo_classic}">
+                    <plugin>gazebo_ros2_control/GazeboSystem</plugin>
+                </xacro:if>
+                <xacro:unless value="${gazebo_classic}">
+                    <plugin>ign_ros2_control/IgnitionSystem</plugin>
+                </xacro:unless>
             </hardware>
             <joint name="J1">
@@ -77,7 +82,15 @@
         <!-- Gazebo plugins -->
         <gazebo>
-            <plugin filename="libgazebo_ros2_control.so" name="gazebo_ros2_control">
-                <parameters>$(find robot_moveit_config)/config/ros2_controllers.yaml</parameters>
-            </plugin>
+            <xacro:if value="${gazebo_classic}">
+                <plugin filename="libgazebo_ros2_control.so" name="gazebo_ros2_control">
+                    <parameters>$(find robot_moveit_config)/config/ros2_controllers.yaml</parameters>
+                </plugin>
+            </xacro:if>
+            <xacro:unless value="${gazebo_classic}">
+                <plugin filename="ign_ros2_control-system" name="ign_ros2_control::IgnitionROS2ControlPlugin">
+                    <parameters>$(find robot_moveit_config)/config/ros2_controllers.yaml</parameters>
+                </plugin>
+                <plugin filename="libignition-gazebo-imu-system.so" name="ignition::gazebo::systems::Imu"/>
+            </xacro:unless>
         </gazebo>
         <!-- Add colours to the robot in Gazebo -->

Commit message: merged all simulation controllers into simulation_interface.xacro

File: robot_description/urdf/robot.xacro (robot description, xacro)
@@ -3,19 +3,12 @@
   <!-- Arguments -->
   <xacro:arg name="moveit_only" default="false"/>
-  <xacro:arg name="gazebo_classic" default="false"/>
+  <xacro:arg name="gazebo_classic" default="true"/>
   <!-- Utils -->
   <xacro:include filename="$(find robot_description)/urdf/utils.xacro" />
   <!-- Robot model-->
   <xacro:include filename="$(find robot_description)/urdf/robot.urdf.xacro"/>
-  <!-- Load Gazebo Controllers unless moveit_only is true -->
-  <xacro:unless value="$(arg moveit_only)">
-    <xacro:include filename="$(find robot_description)/urdf/simulation_interface.xacro"/>
-    <xacro:ros2_control name="GazeboSystem" initial_positions_file="$(find robot_moveit_config)/config/initial_positions.yaml" gazebo_classic="$(arg gazebo_classic)"/>
-  </xacro:unless>
-  <!-- Load MoveIt Controllers if moveit_only is true -->
-  <xacro:if value="$(arg moveit_only)">
-    <xacro:include filename="$(find robot_description)/urdf/moveit_ros2_control.xacro" />
-    <xacro:ros2_control name="FakeSystem" initial_positions_file="$(find robot_moveit_config)/config/initial_positions.yaml"/>
-  </xacro:if>
+  <!-- Simulation interface -->
+  <xacro:include filename="$(find robot_description)/urdf/simulation_interface.xacro"/>
+  <xacro:ros2_control name="GazeboSystem" initial_positions_file="$(find robot_moveit_config)/config/initial_positions.yaml" moveit_only="$(arg moveit_only)" gazebo_classic="$(arg gazebo_classic)"/>
   <xacro:crx10ial/>
 </robot>

File: robot_description/urdf/simulation_interface.xacro (robot description, xacro)
@@ -1,14 +1,21 @@
 <?xml version="1.0"?>
 <robot name="crx10ial" xmlns:xacro="http://www.ros.org/wiki/xacro">
-    <xacro:macro name="ros2_control" params="name initial_positions_file gazebo_classic">
+    <xacro:macro name="ros2_control" params="name initial_positions_file moveit_only gazebo_classic">
         <xacro:property name="initial_positions" value="${xacro.load_yaml(initial_positions_file)['initial_positions']}"/>
         <!-- Simulation ros2_control interface -->
         <ros2_control name="${name}" type="system">
             <hardware>
-                <xacro:if value="${gazebo_classic}">
-                    <plugin>gazebo_ros2_control/GazeboSystem</plugin>
+                <!-- When only MoveIt is loaded, load MoveIt controller -->
+                <xacro:if value="${moveit_only}">
+                    <plugin>mock_components/GenericSystem</plugin>
                 </xacro:if>
-                <xacro:unless value="${gazebo_classic}">
-                    <plugin>ign_ros2_control/IgnitionSystem</plugin>
+                <!-- When Gazebo is also loaded, load Gazebo controllers -->
+                <xacro:unless value="${moveit_only}">
+                    <xacro:if value="${gazebo_classic}">
+                        <plugin>gazebo_ros2_control/GazeboSystem</plugin>
+                    </xacro:if>
+                    <xacro:unless value="${gazebo_classic}">
+                        <plugin>ign_ros2_control/IgnitionSystem</plugin>
+                    </xacro:unless>
                 </xacro:unless>
             </hardware>
