Commit message: file consistency and restructuring between packages

File: robot_description/urdf/gazebo.ros2_control.xacro (robot description, xacro)
@@ -94,4 +94,10 @@
             </joint>
         </ros2_control>
+        <gazebo reference="world" />
+        <gazebo>
+          <plugin filename="libign_ros2_control-system" name="ign_ros2_control::IgnitionROS2ControlPlugin">
+            <parameters>$(find robot_moveit_config)/config/controllers.yaml</parameters>
+          </plugin>
+        </gazebo>
     </xacro:macro>
 </robot>

File: robot_description/urdf/moveit.ros2_control.xacro (robot description, xacro)
@@ -1,9 +1,8 @@
 <?xml version="1.0"?>
 <robot xmlns:xacro="http://www.ros.org/wiki/xacro">
-    <xacro:macro name="crx10ia_l_ros2_control" params="name initial_positions_file">
+    <xacro:macro name="moveit_ros2_control" params="initial_positions_file">
         <xacro:property name="initial_positions" value="${xacro.load_yaml(initial_positions_file)['initial_positions']}"/>
-        <ros2_control name="${name}" type="system">
+        <ros2_control name="crx10ia_l" type="system">
             <hardware>
-                <!-- By default, set up controllers for simulation. This won't work on real hardware -->
                 <plugin>mock_components/GenericSystem</plugin>
             </hardware>

File: robot_description/urdf/robot.gazebo.xacro (robot description, xacro)
@@ -1,18 +1,13 @@
 <?xml version="1.0"?>
 <robot xmlns:xacro="http://wiki.ros.org/xacro" name="crx10ia_l">
-  <xacro:include filename="$(find robot_description)/urdf/robot.xacro" />
-  <xacro:include filename="$(find robot_description)/urdf/gazebo.ros2_control.xacro" />
-  <xacro:arg name="simulation_controllers" default="$(find robot_moveit_config)/config/controllers.yaml" />
-  <xacro:gazebo_ros2_control
-    plugin_name="ign_ros2_control/IgnitionSystem"
-    initial_positions_file="$(find robot_moveit_config)/config/initial_positions.yaml"
-    robot_parameters_file="$(find robot_moveit_config)/config/crx10ia_l.yaml"
-    driver_parameters_file="$(find robot_moveit_config)/config/driver.yaml"
-  />
-  <gazebo reference="world" />
-    <gazebo>
-    <plugin filename="libign_ros2_control-system" name="ign_ros2_control::IgnitionROS2ControlPlugin">
-      <parameters>$(arg simulation_controllers)</parameters>
-    </plugin>
-  </gazebo>
+    <!-- Robot model -->
+    <xacro:include filename="$(find robot_description)/urdf/robot.xacro" />
+    <!-- Gazebo ROS2 Control -->
+    <xacro:include filename="$(find robot_description)/urdf/gazebo.ros2_control.xacro" />
+    <xacro:gazebo_ros2_control
+      plugin_name="ign_ros2_control/IgnitionSystem"
+      initial_positions_file="$(find robot_moveit_config)/config/initial_positions.yaml"
+      robot_parameters_file="$(find robot_moveit_config)/config/crx10ia_l.yaml"
+      driver_parameters_file="$(find robot_moveit_config)/config/driver.yaml"
+    />
 </robot>

File: robot_description/urdf/robot.urdf.xacro (robot description, xacro)
@@ -57,5 +57,5 @@
         <origin xyz="0 0 0" rpy="0 0 0"/>
         <geometry>
-          <mesh filename="file://$(find robot_description)/meshes/crx10ia_l/visual/base.stl" scale="0.001 0.001 0.001"/>
+          <mesh filename="file://$(find robot_description)/meshes/visual/base.stl" scale="0.001 0.001 0.001"/>
         </geometry>
         <material name="FANUC_Black"/>
@@ -64,5 +64,5 @@
         <origin xyz="0 0 0" rpy="0 0 0"/>
         <geometry>
-          <mesh filename="file://$(find robot_description)/meshes/crx10ia_l/collision/base.stl" scale="0.001 0.001 0.001"/>
+          <mesh filename="file://$(find robot_description)/meshes/collision/base.stl" scale="0.001 0.001 0.001"/>
         </geometry>
       </collision>
@@ -84,5 +84,5 @@
         <origin xyz="0 0 ${mz_1 - l_base}" rpy="0 0 0"/>
         <geometry>
-          <mesh filename="file://$(find robot_description)/meshes/crx10ia_l/visual/j1.stl" scale="0.001 0.001 0.001"/>
+          <mesh filename="file://$(find robot_description)/meshes/visual/j1.stl" scale="0.001 0.001 0.001"/>
         </geometry>
         <material name="FANUC_White"/>
@@ -91,5 +91,5 @@
         <origin xyz="0 0 ${mz_1 - l_base}" rpy="0 0 0"/>
         <geometry>
-          <mesh filename="file://$(find robot_description)/meshes/crx10ia_l/collision/j1.stl" scale="0.001 0.001 0.001"/>
+          <mesh filename="file://$(find robot_description)/meshes/collision/j1.stl" scale="0.001 0.001 0.001"/>
         </geometry>
       </collision>
@@ -113,5 +113,5 @@
         <origin xyz="-${l_1} 0 ${mz_2 - l_base}" rpy="0 0 0"/>
         <geometry>
-          <mesh filename="file://$(find robot_description)/meshes/crx10ia_l/visual/j2.stl" scale="0.001 0.001 0.001"/>
+          <mesh filename="file://$(find robot_description)/meshes/visual/j2.stl" scale="0.001 0.001 0.001"/>
         </geometry>
         <material name="FANUC_White"/>
@@ -120,5 +120,5 @@
         <origin xyz="-${l_1} 0 ${mz_2 - l_base}" rpy="0 0 0"/>
         <geometry>
-          <mesh filename="file://$(find robot_description)/meshes/crx10ia_l/collision/j2.stl" scale="0.001 0.001 0.001"/>
+          <mesh filename="file://$(find robot_description)/meshes/collision/j2.stl" scale="0.001 0.001 0.001"/>
         </geometry>
       </collision>
@@ -142,5 +142,5 @@
         <origin xyz="-${l_1} 0 ${mz_3 - l_base - l_2}" rpy="0 0 0"/>
         <geometry>
-          <mesh filename="file://$(find robot_description)/meshes/crx10ia_l/visual/j3.stl" scale="0.001 0.001 0.001"/>
+          <mesh filename="file://$(find robot_description)/meshes/visual/j3.stl" scale="0.001 0.001 0.001"/>
         </geometry>
         <material name="FANUC_White"/>
@@ -149,5 +149,5 @@
         <origin xyz="-${l_1} 0 ${mz_3 - l_base - l_2}" rpy="0 0 0"/>
         <geometry>
-          <mesh filename="file://$(find robot_description)/meshes/crx10ia_l/collision/j3.stl" scale="0.001 0.001 0.001"/>
+          <mesh filename="file://$(find robot_description)/meshes/collision/j3.stl" scale="0.001 0.001 0.001"/>
         </geometry>
       </collision>
@@ -170,5 +170,5 @@
         <origin xyz="${mx_1 - l_1} 0 ${mz_3 - l_base - l_2 - l_3}" rpy="0 0 0"/>
         <geometry>
-          <mesh filename="file://$(find robot_description)/meshes/crx10ia_l/visual/j4.stl" scale="0.001 0.001 0.001"/>
+          <mesh filename="file://$(find robot_description)/meshes/visual/j4.stl" scale="0.001 0.001 0.001"/>
         </geometry>
         <material name="FANUC_White"/>
@@ -177,5 +177,5 @@
         <origin xyz="${mx_1 - l_1} 0 ${mz_3 - l_base - l_2 - l_3}" rpy="0 0 0"/>
         <geometry>
-          <mesh filename="file://$(find robot_description)/meshes/crx10ia_l/collision/j4.stl" scale="0.001 0.001 0.001"/>
+          <mesh filename="file://$(find robot_description)/meshes/collision/j4.stl" scale="0.001 0.001 0.001"/>
         </geometry>
       </collision>
@@ -198,5 +198,5 @@
         <origin xyz="${mx_1 -l_1 - l_4} ${my_1} ${mz_3 - l_base - l_2 - l_3}" rpy="0 0 0"/>
         <geometry>
-          <mesh filename="file://$(find robot_description)/meshes/crx10ia_l/visual/j5.stl" scale="0.001 0.001 0.001"/>
+          <mesh filename="file://$(find robot_description)/meshes/visual/j5.stl" scale="0.001 0.001 0.001"/>
         </geometry>
         <material name="FANUC_White"/>
@@ -205,5 +205,5 @@
         <origin xyz="${mx_1 -l_1 - l_4} ${my_1} ${mz_3 - l_base - l_2 - l_3}" rpy="0 0 0"/>
         <geometry>
-          <mesh filename="file://$(find robot_description)/meshes/crx10ia_l/collision/j5.stl" scale="0.001 0.001 0.001"/>
+          <mesh filename="file://$(find robot_description)/meshes/collision/j5.stl" scale="0.001 0.001 0.001"/>
         </geometry>
       </collision>
@@ -226,5 +226,5 @@
         <origin xyz="${mx_2 -l_1 - l_4} ${my_1 + l_5} ${mz_3 - l_base - l_2 - l_3}" rpy="0 0 0"/>
         <geometry>
-          <mesh filename="file://$(find robot_description)/meshes/crx10ia_l/visual/j6.stl" scale="0.001 0.001 0.001"/>
+          <mesh filename="file://$(find robot_description)/meshes/visual/j6.stl" scale="0.001 0.001 0.001"/>
         </geometry>
 	      <material name="FANUC_Black"/>
@@ -233,5 +233,5 @@
         <origin xyz="${mx_2 -l_1 - l_4} ${my_1 + l_5} ${mz_3 - l_base - l_2 - l_3}" rpy="0 0 0"/>
         <geometry>
-          <mesh filename="file://$(find robot_description)/meshes/crx10ia_l/collision/j6.stl" scale="0.001 0.001 0.001"/>
+          <mesh filename="file://$(find robot_description)/meshes/collision/j6.stl" scale="0.001 0.001 0.001"/>
         </geometry>
       </collision>

File: robot_description/urdf/robot.xacro (robot description, xacro)
@@ -1,9 +1,9 @@
 <?xml version="1.0"?>
 <robot name="crx10ia_l" xmlns:xacro="http://wiki.ros.org/xacro">
-  <!-- Utils -->
-  <!-- <xacro:include filename="$(find robot_description)/urdf/utils.xacro" /> -->
-  <!-- Robot model-->
-  <xacro:include filename="$(find robot_description)/urdf/robot.urdf.xacro"/>
-  <link name="world" />
-  <xacro:crx_robot parent="world"/>
+    <!-- Utils -->
+    <!-- <xacro:include filename="$(find robot_description)/urdf/utils.xacro" /> -->
+    <!-- Robot model-->
+    <xacro:include filename="$(find robot_description)/urdf/robot.urdf.xacro"/>
+    <link name="world" />
+    <xacro:crx_robot parent="world"/>
 </robot>

Commit message: moveit part of test.launch.py is working, Gazebo is still static

File: robot_description/urdf/gazebo.ros2_control.xacro (robot description, xacro)
@@ -1,8 +1,5 @@
 <?xml version="1.0"?>
 <robot xmlns:xacro="http://www.ros.org/wiki/xacro">
-    <xacro:macro name="gazebo_ros2_control" params="
-    plugin_name
-    initial_positions_file
-    ">
+    <xacro:macro name="gazebo_ros2_control" params="initial_positions_file">
         <xacro:property name="initial_positions" value="${xacro.load_yaml(initial_positions_file)['initial_positions']}"/>
         <xacro:property name = "robot_parameters_file" value="$(find robot_description)/config/crx10ia_l.yaml"/>
@@ -10,5 +7,5 @@
         <ros2_control name="crx10ia_l" type="system">
             <hardware>
-                <plugin>${plugin_name}</plugin>
+                <plugin>ign_ros2_control/IgnitionSystem</plugin>
             </hardware>
             <joint name="J1">

File: robot_description/urdf/robot.gazebo.xacro (robot description, xacro)
@@ -6,6 +6,5 @@
     <xacro:include filename="$(find robot_description)/urdf/gazebo.ros2_control.xacro" />
     <xacro:gazebo_ros2_control
-      plugin_name="ign_ros2_control/IgnitionSystem"
-      initial_positions_file="$(find robot_moveit_config)/config/initial_positions.yaml"
+        initial_positions_file="$(find robot_moveit_config)/config/initial_positions.yaml"
     />
 </robot>
