Commit message: experiment with test.launch.py

File: robot_description/urdf/robot.urdf.xacro (robot description, xacro)
@@ -48,5 +48,5 @@
         </geometry>
       </collision>
-      <xacro:cylinder_inertia m="1000.0" r="10.0" h="10.0" /> <!-- Artifically made very heavy to stay in place -->
+      <xacro:cylinder_inertia m="10.0" r="0.05" h="0.1" />
     </link>
     <link name="J1_link">
@@ -64,5 +64,5 @@
         </geometry>
       </collision>
-      <xacro:cylinder_inertia m="10.0" r="10.0" h="10.0" />
+      <xacro:cylinder_inertia m="5.5" r="0.08" h="0.24" />
     </link>
     <link name="J2_link">
@@ -80,5 +80,5 @@
         </geometry>
       </collision>
-      <xacro:cylinder_inertia m="10.0" r="10.0" h="10.0" />
+      <xacro:cylinder_inertia m="12.1" r="0.07" h="0.85" />
     </link>
     <link name="J3_link">
@@ -96,5 +96,5 @@
         </geometry>
       </collision>
-      <xacro:cylinder_inertia m="10.0" r="10.0" h="10.0" />
+      <xacro:cylinder_inertia m="2.8" r="0.06" h="0.23" />
     </link>
     <link name="J4_link">
@@ -112,5 +112,5 @@
         </geometry>
       </collision>
-      <xacro:cylinder_inertia m="10.0" r="10.0" h="10.0" />
+      <xacro:cylinder_inertia m="3.4" r="0.05" h="0.42" />
     </link>
     <link name="J5_link">
@@ -128,5 +128,5 @@
         </geometry>
       </collision>
-      <xacro:cylinder_inertia m="10.0" r="10.0" h="10.0" />
+      <xacro:cylinder_inertia m="1.5" r="0.05" h="0.16" />
     </link>
     <link name="J6_link">
@@ -144,5 +144,5 @@
         </geometry>
       </collision>
-      <xacro:cylinder_inertia m="10.0" r="10.0" h="10.0" />
+      <xacro:cylinder_inertia m="0.5" r="0.04" h="0.06" />
     </link>
     <!-- joints -->
@@ -152,5 +152,6 @@
       <child link="J1_link"/>
       <axis xyz="0 0 1"/>
-      <limit lower="${j1_l * pi / 180}" upper="${j1_u * pi / 180}" effort="0" velocity="${j1_v * pi / 180}"/>
+      <limit lower="${j1_l * pi / 180}" upper="${j1_u * pi / 180}" effort="50" velocity="${j1_v * pi / 180}"/>
+      <dynamics damping="0.1" friction="0.3"/>
     </joint>
     <joint name="J2" type="revolute">
@@ -159,5 +160,6 @@
       <child link="J2_link"/>
       <axis xyz="0 1 0"/>
-      <limit lower="${j2_l * pi / 180}" upper="${j2_u * pi / 180}" effort="0" velocity="${j2_v * pi / 180}"/>
+      <limit lower="${j2_l * pi / 180}" upper="${j2_u * pi / 180}" effort="50" velocity="${j2_v * pi / 180}"/>
+      <dynamics damping="0.1" friction="0.2"/>
     </joint>
     <joint name="J3" type="revolute">
@@ -166,5 +168,6 @@
       <child link="J3_link"/>
       <axis xyz="0 -1 0"/>
-      <limit lower="${j3_l * pi / 180}" upper="${j3_u * pi / 180}" effort="0" velocity="${j3_v * pi / 180}"/>
+      <limit lower="${j3_l * pi / 180}" upper="${j3_u * pi / 180}" effort="50" velocity="${j3_v * pi / 180}"/>
+      <dynamics damping="0.1" friction="0.2"/>
     </joint>
     <joint name="J4" type="revolute">
@@ -173,5 +176,6 @@
       <child link="J4_link"/>
       <axis xyz="-1 0 0"/>
-      <limit lower="${j4_l * pi / 180}" upper="${j4_u * pi / 180}" effort="0" velocity="${j4_v * pi / 180}"/>
+      <limit lower="${j4_l * pi / 180}" upper="${j4_u * pi / 180}" effort="50" velocity="${j4_v * pi / 180}"/>
+      <dynamics damping="0.1" friction="0.1"/>
     </joint>
     <joint name="J5" type="revolute">
@@ -180,5 +184,6 @@
       <child link="J5_link"/>
       <axis xyz="0 -1 0"/>
-      <limit lower="${j5_l * pi / 180}" upper="${j5_u * pi / 180}" effort="0" velocity="${j5_v * pi / 180}"/>
+      <limit lower="${j5_l * pi / 180}" upper="${j5_u * pi / 180}" effort="50" velocity="${j5_v * pi / 180}"/>
+      <dynamics damping="0.1" friction="0.1"/>
     </joint>
     <joint name="J6" type="revolute">
@@ -187,5 +192,6 @@
       <child link="J6_link"/>
       <axis xyz="-1 0 0"/>
-      <limit lower="${j6_l * pi / 180}" upper="${j6_u * pi / 180}" effort="0" velocity="${j6_v * pi / 180}"/>
+      <limit lower="${j6_l * pi / 180}" upper="${j6_u * pi / 180}" effort="50" velocity="${j6_v * pi / 180}"/>
+      <dynamics damping="0.1" friction="0.01"/>
     </joint>
     <joint name="imu_joint" type="fixed">

File: robot_description/urdf/simulation_interface.xacro (robot description, xacro)
@@ -19,4 +19,8 @@
                 </state_interface>
                 <state_interface name="velocity"/>
+                <state_interface name="effort"/>
+                <ros2_control>
+                    <hardwareInterface>hardware_interface/PositionJointInterface</hardwareInterface>
+                </ros2_control>
             </joint>
             <joint name="J2">
@@ -29,4 +33,8 @@
                 </state_interface>
                 <state_interface name="velocity"/>
+                <state_interface name="effort"/>
+                <ros2_control>
+                    <hardwareInterface>hardware_interface/PositionJointInterface</hardwareInterface>
+                </ros2_control>
             </joint>
             <joint name="J3">
@@ -39,4 +47,8 @@
                 </state_interface>
                 <state_interface name="velocity"/>
+                <state_interface name="effort"/>
+                <ros2_control>
+                    <hardwareInterface>hardware_interface/PositionJointInterface</hardwareInterface>
+                </ros2_control>
             </joint>
             <joint name="J4">
@@ -49,4 +61,8 @@
                 </state_interface>
                 <state_interface name="velocity"/>
+                <state_interface name="effort"/>
+                <ros2_control>
+                    <hardwareInterface>hardware_interface/PositionJointInterface</hardwareInterface>
+                </ros2_control>
             </joint>
             <joint name="J5">
@@ -59,4 +75,8 @@
                 </state_interface>
                 <state_interface name="velocity"/>
+                <state_interface name="effort"/>
+                <ros2_control>
+                    <hardwareInterface>hardware_interface/PositionJointInterface</hardwareInterface>
+                </ros2_control>
             </joint>
             <joint name="J6">
@@ -69,4 +89,8 @@
                 </state_interface>
                 <state_interface name="velocity"/>
+                <state_interface name="effort"/>
+                <ros2_control>
+                    <hardwareInterface>hardware_interface/PositionJointInterface</hardwareInterface>
+                </ros2_control>
             </joint>
         </ros2_control>
@@ -78,5 +102,14 @@
             </plugin>
             <plugin filename="libgazebo_ros2_control.so" name="gazebo_ros2_control">
-                <robotNamespace>/</robotNamespace>
+                <!-- Set the ROS 2 namespace for the robot -->
+                <robotNamespace>/robot</robotNamespace>
+                <!-- Path to the robot's hardware interface -->
+                <parameters>$(find robot_moveit_config)/config/controller_params.yaml</parameters>
+                <!-- Enable or disable publishing joint states -->
+                <publishRate>50</publishRate> <!-- Publish joint states at 50 Hz -->
+                <!-- Update rate for control (usually matches simulation update rate) -->
+                <controlPeriod>0.001</controlPeriod> <!-- Control loop period in seconds -->
+                <!-- Whether to publish the joint states (default is true) -->
+                <publishJointStates>false</publishJointStates>
             </plugin>
             <!-- IMU -->
@@ -87,14 +120,4 @@
             </plugin>
         </gazebo>
-        <!-- Sensor simulation -->
-        <gazebo reference="imu_link">
-            <sensor name="imu" type="imu">
-                <always_on>1</always_on>
-                <update_rate>15</update_rate>
-                <visualize>false</visualize>
-                <topic>imu/data</topic>
-                <ignition_frame_id>imu_link</ignition_frame_id>
-            </sensor>
-        </gazebo>
     </xacro:macro>
 </robot>

Commit message: gazebo classic WORKS!

File: robot_description/urdf/robot.urdf.xacro (robot description, xacro)
@@ -48,5 +48,9 @@
         </geometry>
       </collision>
-      <xacro:cylinder_inertia m="10.0" r="0.05" h="0.1" />
+      <inertial>
+        <mass value="9.0" />
+        <origin xyz="0 0 0" rpy="0 0 0" />
+        <inertia ixx="0.095" ixy="0" ixz="0" iyy="0.095" iyz="0" izz="0.36" />
+      </inertial>
     </link>
     <link name="J1_link">
@@ -64,5 +68,9 @@
         </geometry>
       </collision>
-      <xacro:cylinder_inertia m="5.5" r="0.08" h="0.24" />
+      <inertial>
+        <mass value="5.0" />
+        <origin xyz="0 0 0" rpy="0 0 0" />
+        <inertia ixx="0.033" ixy="0" ixz="0" iyy="0.033" iyz="0" izz="0.0075" />
+      </inertial>
     </link>
     <link name="J2_link">
@@ -80,5 +88,9 @@
         </geometry>
       </collision>
-      <xacro:cylinder_inertia m="12.1" r="0.07" h="0.85" />
+      <inertial>
+        <mass value="8.0" />
+        <origin xyz="0 0 0" rpy="0 0 0" />
+        <inertia ixx="0.500" ixy="0" ixz="0" iyy="0.500" iyz="0" izz="0.020" />
+      </inertial>
     </link>
     <link name="J3_link">
@@ -96,5 +108,9 @@
         </geometry>
       </collision>
-      <xacro:cylinder_inertia m="2.8" r="0.06" h="0.23" />
+      <inertial>
+        <mass value="4.0" />
+        <origin xyz="0 0 0" rpy="0 0 0" />
+        <inertia ixx="0.025" ixy="0" ixz="0" iyy="0.025" iyz="0" izz="0.005" />
+      </inertial>
     </link>
     <link name="J4_link">
@@ -112,5 +128,9 @@
         </geometry>
       </collision>
-      <xacro:cylinder_inertia m="3.4" r="0.05" h="0.42" />
+      <inertial>
+        <mass value="5.0" />
+        <origin xyz="0 0 0" rpy="0 0 0" />
+        <inertia ixx="0.080" ixy="0" ixz="0" iyy="0.080" iyz="0" izz="0.010" />
+      </inertial>
     </link>
     <link name="J5_link">
@@ -128,5 +148,9 @@
         </geometry>
       </collision>
-      <xacro:cylinder_inertia m="1.5" r="0.05" h="0.16" />
+      <inertial>
+        <mass value="3.0" />
+        <origin xyz="0 0 0" rpy="0 0 0" />
+        <inertia ixx="0.010" ixy="0" ixz="0" iyy="0.010" iyz="0" izz="0.004" />
+      </inertial>
     </link>
     <link name="J6_link">
@@ -144,5 +168,9 @@
         </geometry>
       </collision>
-      <xacro:cylinder_inertia m="0.5" r="0.04" h="0.06" />
+      <inertial>
+        <mass value="2.0" />
+        <origin xyz="0 0 0" rpy="0 0 0" />
+        <inertia ixx="0.001" ixy="0" ixz="0" iyy="0.001" iyz="0" izz="0.0005" />
+      </inertial>
     </link>
     <!-- joints -->

File: robot_description/urdf/robot.xacro (robot description, xacro)
@@ -5,6 +5,6 @@
   <!-- Robot model-->
   <xacro:include filename="$(find robot_description)/urdf/robot.urdf.xacro"/>
-  <!-- Simulation interface -->
-  <xacro:include filename="$(find robot_description)/urdf/simulation_interface.xacro" />
+  <!-- Simulation interface, located in MoveIt package-->
+  <xacro:include filename = "$(find robot_description)/urdf/simulation_interface.xacro" />
   <xacro:crx10ial/>
 </robot>

File: robot_description/urdf/simulation_interface.xacro (robot description, xacro)
@@ -1,106 +1,82 @@
 <?xml version="1.0"?>
-<robot xmlns:xacro="http://www.ros.org/wiki/xacro">
-    <xacro:macro name="crx10ial_ros2_control" params="name initial_positions_file">
-        <xacro:property name="initial_positions" value="${load_yaml(initial_positions_file)['initial_positions']}"/>
-        <!-- Simulation ros2_control interface -->
-        <!--<ros2_control name="${name}" type="system">-->
-        <ros2_control name="GazeboSystem" type="system"> <!-- Replaced ${name} with GazeboSimSystem-->
-            <hardware>
-                <!-- By default, set up controllers for simulation. This won't work on real hardware -->
-                <!-- <plugin>mock_components/GenericSystem</plugin> -->
-                <!-- <plugin>ign_ros2_control/IgnitionSystem</plugin> -->
-                <plugin>gazebo_ros2_control/GazeboSystem</plugin>
-            </hardware>
-            <joint name="J1">
-                <command_interface name="position">
-                    <param name="min">{-2*pi}</param>
-                    <param name="max">{2*pi}</param>
-                </command_interface>
-                <state_interface name="position">
-                  <param name="initial_value">${initial_positions['J1']}</param>
-                </state_interface>
-                <state_interface name="velocity"/>
-                <state_interface name="effort"/>
-                <ros2_control>
-                    <hardwareInterface>hardware_interface/PositionJointInterface</hardwareInterface>
-                </ros2_control>
-            </joint>
-            <joint name="J2">
-                <command_interface name="position">
-                    <param name="min">{-2*pi}</param>
-                    <param name="max">{2*pi}</param>
-                </command_interface>
-                <state_interface name="position">
-                  <param name="initial_value">${initial_positions['J2']}</param>
-                </state_interface>
-                <state_interface name="velocity"/>
-                <state_interface name="effort"/>
-                <ros2_control>
-                    <hardwareInterface>hardware_interface/PositionJointInterface</hardwareInterface>
-                </ros2_control>
-            </joint>
-            <joint name="J3">
-                <command_interface name="position">
-                    <param name="min">{pi}</param>
-                    <param name="max">{pi}</param>
-                </command_interface>
-                <state_interface name="position">
-                  <param name="initial_value">${initial_positions['J3']}</param>
-                </state_interface>
-                <state_interface name="velocity"/>
-                <state_interface name="effort"/>
-                <ros2_control>
-                    <hardwareInterface>hardware_interface/PositionJointInterface</hardwareInterface>
-                </ros2_control>
-            </joint>
-            <joint name="J4">
-                <command_interface name="position">
-                    <param name="min">{-2*pi}</param>
-                    <param name="max">{2*pi}</param>
-                </command_interface>
-                <state_interface name="position">
-                  <param name="initial_value">${initial_positions['J4']}</param>
-                </state_interface>
-                <state_interface name="velocity"/>
-                <state_interface name="effort"/>
-                <ros2_control>
-                    <hardwareInterface>hardware_interface/PositionJointInterface</hardwareInterface>
-                </ros2_control>
-            </joint>
-            <joint name="J5">
-                <command_interface name="position">
-                    <param name="min">{-2*pi}</param>
-                    <param name="max">{2*pi}</param>
-                </command_interface>
-                <state_interface name="position">
-                  <param name="initial_value">${initial_positions['J5']}</param>
-                </state_interface>
-                <state_interface name="velocity"/>
-                <state_interface name="effort"/>
-                <ros2_control>
-                    <hardwareInterface>hardware_interface/PositionJointInterface</hardwareInterface>
-                </ros2_control>
-            </joint>
-            <joint name="J6">
-                <command_interface name="position">
-                    <param name="min">{-2*pi}</param>
-                    <param name="max">{2*pi}</param>
-                </command_interface>
-                <state_interface name="position">
-                  <param name="initial_value">${initial_positions['J6']}</param>
-                </state_interface>
-                <state_interface name="velocity"/>
-                <state_interface name="effort"/>
-                <ros2_control>
-                    <hardwareInterface>hardware_interface/PositionJointInterface</hardwareInterface>
-                </ros2_control>
-            </joint>
-        </ros2_control>
-        <!-- Gazebo plugins -->
-        <gazebo>
-            <plugin name="gazebo_ros2_control" filename="libgazebo_ros2_control.so">
-                <parameters>$(find robot_moveit_config)/config/ros2_controllers.yaml</parameters>
-            </plugin>
-        </gazebo>
-    </xacro:macro>
+<robot name="crx10ial" xmlns:xacro="http://www.ros.org/wiki/xacro">
+    <!-- Simulation ros2_control interface -->
+    <ros2_control name="GazeboSystem" type="system">
+        <hardware>
+            <plugin>gazebo_ros2_control/GazeboSystem</plugin>
+        </hardware>
+        <joint name="J1">
+            <command_interface name="position">
+                <param name="min">{-2*pi}</param>
+                <param name="max">{2*pi}</param>
+            </command_interface>
+            <state_interface name="position">
+            <param name="initial_value">0</param>
+            </state_interface>
+            <state_interface name="velocity"/>
+            <state_interface name="effort"/>
+        </joint>
+        <joint name="J2">
+            <command_interface name="position">
+                <param name="min">{-2*pi}</param>
+                <param name="max">{2*pi}</param>
+            </command_interface>
+            <state_interface name="position">
+            <param name="initial_value">0</param>
+            </state_interface>
+            <state_interface name="velocity"/>
+            <state_interface name="effort"/>
+        </joint>
+        <joint name="J3">
+            <command_interface name="position">
+                <param name="min">{pi}</param>
+                <param name="max">{pi}</param>
+            </command_interface>
+            <state_interface name="position">
+            <param name="initial_value">0</param>
+            </state_interface>
+            <state_interface name="velocity"/>
+            <state_interface name="effort"/>
+        </joint>
+        <joint name="J4">
+            <command_interface name="position">
+                <param name="min">{-2*pi}</param>
+                <param name="max">{2*pi}</param>
+            </command_interface>
+            <state_interface name="position">
+            <param name="initial_value">0</param>
+            </state_interface>
+            <state_interface name="velocity"/>
+            <state_interface name="effort"/>
+        </joint>
+        <joint name="J5">
+            <command_interface name="position">
+                <param name="min">{-2*pi}</param>
+                <param name="max">{2*pi}</param>
+            </command_interface>
+            <state_interface name="position">
+            <param name="initial_value">0</param>
+            </state_interface>
+            <state_interface name="velocity"/>
+            <state_interface name="effort"/>
+        </joint>
+        <joint name="J6">
+            <command_interface name="position">
+                <param name="min">{-2*pi}</param>
+                <param name="max">{2*pi}</param>
+            </command_interface>
+            <state_interface name="position">
+            <param name="initial_value">0</param>
+            </state_interface>
+            <state_interface name="velocity"/>
+            <state_interface name="effort"/>
+        </joint>
+    </ros2_control>
+    <!-- Gazebo plugins -->
+    <gazebo>
+        <!-- ros2_control -->
+        <plugin filename="libgazebo_ros2_control.so" name="gazebo_ros2_control">
+            <parameters>$(find robot_moveit_config)/config/ros2_controllers.yaml</parameters>
+        </plugin>
+    </gazebo>
 </robot>

File: robot_moveit_config/config/crx10ial.urdf.xacro (robot description, xacro)
@@ -1,7 +1,6 @@
 <?xml version="1.0"?>
 <robot xmlns:xacro="http://www.ros.org/wiki/xacro" name="crx10ial">
-    <xacro:arg name="initial_positions_file" default="initial_positions.yaml" />
     <!-- Import crx10ial urdf file -->
     <xacro:include filename="$(find robot_description)/urdf/robot.xacro" />
-    <xacro:crx10ial_ros2_control name="IgnitionSystem" initial_positions_file="$(arg initial_positions_file)"/>
+    <xacro:crx10ial_ros2_control name="GazeboSystem" initial_positions_file="$(arg initial_positions_file)"/>
 </robot>
