Commit message: gazebo works, moveit doesnt

File: robot_description/urdf/robot.urdf.xacro (robot description, xacro)
@@ -1,4 +1,4 @@
 <?xml version="1.0"?>
-<robot xmlns:xacro="http://wiki.ros.org/xacro">
+<robot xmlns:xacro="http://wiki.ros.org/xacro" xmlns="http://www.w3.org/2001/XMLSchema-instance">
   <xacro:macro name="crx10ial">
     <xacro:property name="l_base" value="0.245"/>
@@ -48,9 +48,5 @@
         </geometry>
       </collision>
-      <inertial>
-        <mass value="9.0" />
-        <origin xyz="0 0 0" rpy="0 0 0" />
-        <inertia ixx="0.095" ixy="0" ixz="0" iyy="0.095" iyz="0" izz="0.36" />
-      </inertial>
+      <xacro:cylinder_inertia m="10.0" r="0.05" h="0.1" />
     </link>
     <link name="J1_link">
@@ -68,9 +64,5 @@
         </geometry>
       </collision>
-      <inertial>
-        <mass value="5.0" />
-        <origin xyz="0 0 0" rpy="0 0 0" />
-        <inertia ixx="0.033" ixy="0" ixz="0" iyy="0.033" iyz="0" izz="0.0075" />
-      </inertial>
+      <xacro:cylinder_inertia m="5.5" r="0.08" h="0.24" />
     </link>
     <link name="J2_link">
@@ -88,9 +80,5 @@
         </geometry>
       </collision>
-      <inertial>
-        <mass value="8.0" />
-        <origin xyz="0 0 0" rpy="0 0 0" />
-        <inertia ixx="0.500" ixy="0" ixz="0" iyy="0.500" iyz="0" izz="0.020" />
-      </inertial>
+      <xacro:cylinder_inertia m="12.1" r="0.07" h="0.85" />
     </link>
     <link name="J3_link">
@@ -108,9 +96,5 @@
         </geometry>
       </collision>
-      <inertial>
-        <mass value="4.0" />
-        <origin xyz="0 0 0" rpy="0 0 0" />
-        <inertia ixx="0.025" ixy="0" ixz="0" iyy="0.025" iyz="0" izz="0.005" />
-      </inertial>
+      <xacro:cylinder_inertia m="2.8" r="0.06" h="0.23" />
     </link>
     <link name="J4_link">
@@ -128,9 +112,5 @@
         </geometry>
       </collision>
-      <inertial>
-        <mass value="5.0" />
-        <origin xyz="0 0 0" rpy="0 0 0" />
-        <inertia ixx="0.080" ixy="0" ixz="0" iyy="0.080" iyz="0" izz="0.010" />
-      </inertial>
+      <xacro:cylinder_inertia m="3.4" r="0.05" h="0.42" />
     </link>
     <link name="J5_link">
@@ -148,9 +128,5 @@
         </geometry>
       </collision>
-      <inertial>
-        <mass value="3.0" />
-        <origin xyz="0 0 0" rpy="0 0 0" />
-        <inertia ixx="0.010" ixy="0" ixz="0" iyy="0.010" iyz="0" izz="0.004" />
-      </inertial>
+      <xacro:cylinder_inertia m="1.5" r="0.05" h="0.16" />
     </link>
     <link name="J6_link">
@@ -168,9 +144,5 @@
         </geometry>
       </collision>
-      <inertial>
-        <mass value="2.0" />
-        <origin xyz="0 0 0" rpy="0 0 0" />
-        <inertia ixx="0.001" ixy="0" ixz="0" iyy="0.001" iyz="0" izz="0.0005" />
-      </inertial>
+      <xacro:cylinder_inertia m="0.5" r="0.04" h="0.06" />
     </link>
     <!-- joints -->
@@ -235,11 +207,4 @@
       <child link="wbase"/>
     </joint>
-    <!-- Gazebo world attach Doet niks-->
-    <link name="world" />
-    <joint name="world_to_base" type="fixed">
-      <origin xyz="0 0 0" rpy="0 0 0"/>
-      <parent link="world"/>
-      <child link="base_link"/>
-    </joint>
     <!-- flange coords -->
     <link name="flange" />

File: robot_description/urdf/robot.xacro (robot description, xacro)
@@ -5,6 +5,5 @@
   <!-- Robot model-->
   <xacro:include filename="$(find robot_description)/urdf/robot.urdf.xacro"/>
-  <!-- Simulation interface, located in MoveIt package-->
-  <xacro:include filename="$(find robot_description)/urdf/simulation_interface.xacro" />
+  <xacro:include filename="$(find robot_description)/urdf/simulation_interface.xacro"/>
   <xacro:crx10ial/>
 </robot>

File: robot_moveit_config/config/crx10ial.urdf.xacro (robot description, xacro)
@@ -3,4 +3,6 @@
     <!-- Import crx10ial urdf file -->
     <xacro:include filename="$(find robot_description)/urdf/robot.xacro" />
-    <!-- <xacro:crx10ial_ros2_control name="GazeboSystem" initial_positions_file="$(arg initial_positions_file)"/> -->
+    <!-- Import control_xacro -->
+    <xacro:include filename="$(find robot_moveit_config)/config/crx10ial.ros2_control.xacro" />
+    <xacro:crx10ial/>
 </robot>

Commit message: added soft grippers as end effector

File: robot_description/urdf/robot.urdf.xacro (robot description, xacro)
@@ -244,4 +244,6 @@
     <!-- Sensor links (not visualised) -->
     <link name="imu_link"/>
+    <!-- Add soft gripper to end of arm -->
+    <xacro:include filename="$(find robot_description)/urdf/softgripper.urdf.xacro"/>
   </xacro:macro>
 </robot>

File: robot_description/urdf/simulation_interface.xacro (robot description, xacro)
@@ -103,4 +103,23 @@
             <material>Gazebo/Black</material>
         </gazebo>
+        <!-- Add colours to the end effector -->
+        <gazebo reference="quick_changer">
+            <material>Gazebo/Blue</material>
+        </gazebo>
+        <gazebo reference="mounting_plate">
+            <material>Gazebo/Grey</material>
+        </gazebo>
+        <gazebo reference="finger_1">
+            <material>Gazebo/BlueGlow</material>
+        </gazebo>
+        <gazebo reference="finger_2">
+            <material>Gazebo/BlueGlow</material>
+        </gazebo>
+        <gazebo reference="finger_3">
+            <material>Gazebo/BlueGlow</material>
+        </gazebo>
+        <gazebo reference="finger_4">
+            <material>Gazebo/BlueGlow</material>
+        </gazebo>
     </xacro:macro>
 </robot>

File: robot_description/urdf/utils.xacro (robot description, xacro)
@@ -13,4 +13,13 @@
   <material name="FANUC_White">
     <color rgba="0.84 0.84 0.82 1"/>
+  </material>
+  <material name="steel_material">
+    <color rgba="0.7 0.7 0.7 1"/>
+  </material>
+  <material name="blue_material">
+    <color rgba="0.2 0.4 1 1"/>
+  </material>
+    <material name="softgripper">
+    <color rgba="0.3 0.7 1 1"/>
   </material>
   <!-- Inertia macros -->

Commit message: simplified robot urdf

File: robot_description/urdf/robot.urdf.xacro (robot description, xacro)
@@ -2,36 +2,5 @@
 <robot xmlns:xacro="http://wiki.ros.org/xacro" xmlns="http://www.w3.org/2001/XMLSchema-instance">
   <xacro:macro name="crx10ial">
-    <xacro:property name="l_base" value="0.245"/>
-    <xacro:property name="l_1" value="0.0"/>
-    <xacro:property name="l_2" value="0.710"/> <!--Was 0.540, adding (mz_3 new - old) gives new value-->
-    <xacro:property name="l_3" value="0.0"/>
-    <xacro:property name="l_4" value="0.540"/>
-    <xacro:property name="l_5" value="0.150"/>
-    <xacro:property name="l_6" value="0.160"/>
-    <xacro:property name="j1_v" value="120"/>
-    <xacro:property name="j2_v" value="120"/>
-    <xacro:property name="j3_v" value="180"/>
-    <xacro:property name="j4_v" value="180"/>
-    <xacro:property name="j5_v" value="180"/>
-    <xacro:property name="j6_v" value="180"/>
-    <xacro:property name="j1_u" value="190"/>
-    <xacro:property name="j2_u" value="179.9"/>
-    <xacro:property name="j3_u" value="251"/>
-    <xacro:property name="j4_u" value="190"/>
-    <xacro:property name="j5_u" value="179.9"/>
-    <xacro:property name="j6_u" value="225"/>
-    <xacro:property name="j1_l" value="-190"/>
-    <xacro:property name="j2_l" value="-179.9"/>
-    <xacro:property name="j3_l" value="-71"/>
-    <xacro:property name="j4_l" value="-190"/>
-    <xacro:property name="j5_l" value="-179.9"/>
-    <xacro:property name="j6_l" value="-225"/>
-    <xacro:property name="mz_1" value="0.1277"/>
-    <xacro:property name="mz_2" value="0.245"/>
-    <xacro:property name="mz_3" value="0.955"/> <!--Was 0.785-->
-    <xacro:property name="mx_1" value="0.540"/>
-    <xacro:property name="mx_2" value="0.700"/>
-    <xacro:property name="my_1" value="-0.150"/>
-    <!-- links -->
+    <!-- Links -->
     <link name="base_link">
       <visual>
@@ -52,5 +21,5 @@
     <link name="J1_link">
       <visual>
-        <origin xyz="0 0 ${mz_1 - l_base}" rpy="0 0 0"/>
+        <origin xyz="0 0 -0.1173" rpy="0 0 0"/>
         <geometry>
           <mesh filename="file://$(find robot_description)/meshes/visual/j1.stl" scale="0.001 0.001 0.001"/>
@@ -59,5 +28,5 @@
       </visual>
       <collision>
-        <origin xyz="0 0 ${mz_1 - l_base}" rpy="0 0 0"/>
+        <origin xyz="0 0 -0.1173" rpy="0 0 0"/>
         <geometry>
           <mesh filename="file://$(find robot_description)/meshes/collision/j1.stl" scale="0.001 0.001 0.001"/>
@@ -68,5 +37,5 @@
     <link name="J2_link">
       <visual>
-        <origin xyz="-${l_1} 0 ${mz_2 - l_base}" rpy="0 0 0"/>
+        <origin xyz="0 0 0" rpy="0 0 0"/>
         <geometry>
           <mesh filename="file://$(find robot_description)/meshes/visual/j2.stl" scale="0.001 0.001 0.001"/>
@@ -75,5 +44,5 @@
       </visual>
       <collision>
-        <origin xyz="-${l_1} 0 ${mz_2 - l_base}" rpy="0 0 0"/>
+        <origin xyz="0 0 0" rpy="0 0 0"/>
         <geometry>
           <mesh filename="file://$(find robot_description)/meshes/collision/j2.stl" scale="0.001 0.001 0.001"/>
@@ -84,5 +53,5 @@
     <link name="J3_link">
       <visual>
-	      <origin xyz="-${l_1} 0 ${mz_3 - l_base - l_2}" rpy="0 0 0"/>
+	      <origin xyz="0 0 0" rpy="0 0 0"/>
         <geometry>
           <mesh filename="file://$(find robot_description)/meshes/visual/j3.stl" scale="0.001 0.001 0.001"/>
@@ -91,5 +60,5 @@
       </visual>
       <collision>
-        <origin xyz="-${l_1} 0 ${mz_3 - l_base - l_2}" rpy="0 0 0"/>
+        <origin xyz="0 0 0" rpy="0 0 0"/>
         <geometry>
           <mesh filename="file://$(find robot_description)/meshes/collision/j3.stl" scale="0.001 0.001 0.001"/>
@@ -100,5 +69,5 @@
     <link name="J4_link">
       <visual>
-	      <origin xyz="${mx_1 - l_1} 0 ${mz_3 - l_base - l_2 - l_3}" rpy="0 0 0"/>
+	      <origin xyz="0.54 0 0" rpy="0 0 0"/>
         <geometry>
           <mesh filename="file://$(find robot_description)/meshes/visual/j4.stl" scale="0.001 0.001 0.001"/>
@@ -107,5 +76,5 @@
       </visual>
       <collision>
-        <origin xyz="${mx_1 - l_1} 0 ${mz_3 - l_base - l_2 - l_3}" rpy="0 0 0"/>
+        <origin xyz="0.54 0 0" rpy="0 0 0"/>
         <geometry>
           <mesh filename="file://$(find robot_description)/meshes/collision/j4.stl" scale="0.001 0.001 0.001"/>
@@ -116,5 +85,5 @@
     <link name="J5_link">
       <visual>
-        <origin xyz="${mx_1 -l_1 - l_4} ${my_1} ${mz_3 - l_base - l_2 - l_3}" rpy="0 0 0"/>
+        <origin xyz="0 -0.15 0" rpy="0 0 0"/>
         <geometry>
           <mesh filename="file://$(find robot_description)/meshes/visual/j5.stl" scale="0.001 0.001 0.001"/>
@@ -123,5 +92,5 @@
       </visual>
       <collision>
-        <origin xyz="${mx_1 -l_1 - l_4} ${my_1} ${mz_3 - l_base - l_2 - l_3}" rpy="0 0 0"/>
+        <origin xyz="0 -0.150 0" rpy="0 0 0"/>
         <geometry>
           <mesh filename="file://$(find robot_description)/meshes/collision/j5.stl" scale="0.001 0.001 0.001"/>
@@ -132,5 +101,5 @@
     <link name="J6_link">
       <visual>
-        <origin xyz="${mx_2 -l_1 - l_4} ${my_1 + l_5} ${mz_3 - l_base - l_2 - l_3}" rpy="0 0 0"/>
+        <origin xyz="0.16 0 0" rpy="0 0 0"/>
         <geometry>
           <mesh filename="file://$(find robot_description)/meshes/visual/j6.stl" scale="0.001 0.001 0.001"/>
@@ -139,5 +108,5 @@
       </visual>
       <collision>
-        <origin xyz="${mx_2 -l_1 - l_4} ${my_1 + l_5} ${mz_3 - l_base - l_2 - l_3}" rpy="0 0 0"/>
+        <origin xyz="0.16 0 0" rpy="0 0 0"/>
         <geometry>
           <mesh filename="file://$(find robot_description)/meshes/collision/j6.stl" scale="0.001 0.001 0.001"/>
@@ -146,102 +115,60 @@
       <xacro:cylinder_inertia m="0.5" r="0.04" h="0.06" />
     </link>
-    <!-- joints -->
+    <!-- Joints -->
     <joint name="J1" type="revolute">
-      <origin xyz="0 0 ${l_base}" rpy="0 0 0"/>
+      <origin xyz="0 0 0.245" rpy="0 0 0"/>
       <parent link="base_link"/>
       <child link="J1_link"/>
       <axis xyz="0 0 1"/>
-      <limit lower="${j1_l * pi / 180}" upper="${j1_u * pi / 180}" effort="50" velocity="${j1_v * pi / 180}"/>
+      <limit lower="-3.3161" upper="3.3161" effort="50" velocity="2.0944"/>
       <dynamics damping="0.1" friction="0.3"/>
     </joint>
     <joint name="J2" type="revolute">
-      <origin xyz="${l_1} 0 0" rpy="0 0 0"/>
+      <origin xyz="0 0 0" rpy="0 0 0"/>
       <parent link="J1_link"/>
       <child link="J2_link"/>
       <axis xyz="0 1 0"/>
-      <limit lower="${j2_l * pi / 180}" upper="${j2_u * pi / 180}" effort="50" velocity="${j2_v * pi / 180}"/>
+      <limit lower="-3.1398" upper="3.1398" effort="50" velocity="2.0944"/>
       <dynamics damping="0.1" friction="0.2"/>
     </joint>
     <joint name="J3" type="revolute">
-      <origin xyz="0 0 ${l_2}" rpy="0 0 0"/>
+      <origin xyz="0 0 0.71" rpy="0 0 0"/>
       <parent link="J2_link"/>
       <child link="J3_link"/>
       <axis xyz="0 -1 0"/>
-      <limit lower="${j3_l * pi / 180}" upper="${j3_u * pi / 180}" effort="50" velocity="${j3_v * pi / 180}"/>
+      <limit lower="-1.2392" upper="4.3867" effort="50" velocity="3.1416"/>
       <dynamics damping="0.1" friction="0.2"/>
     </joint>
     <joint name="J4" type="revolute">
-      <origin xyz="0 0 ${l_3}" rpy="0 0 0"/>
+      <origin xyz="0 0 0" rpy="0 0 0"/>
       <parent link="J3_link"/>
       <child link="J4_link"/>
       <axis xyz="-1 0 0"/>
-      <limit lower="${j4_l * pi / 180}" upper="${j4_u * pi / 180}" effort="50" velocity="${j4_v * pi / 180}"/>
+      <limit lower="-3.3161" upper="3.3161" effort="50" velocity="3.1416"/>
       <dynamics damping="0.1" friction="0.1"/>
     </joint>
     <joint name="J5" type="revolute">
-      <origin xyz="${l_4} 0 0" rpy="0 0 0"/>
+      <origin xyz="0.54 0 0" rpy="0 0 0"/>
       <parent link="J4_link"/>
       <child link="J5_link"/>
       <axis xyz="0 -1 0"/>
-      <limit lower="${j5_l * pi / 180}" upper="${j5_u * pi / 180}" effort="50" velocity="${j5_v * pi / 180}"/>
+      <limit lower="-3.1398" upper="3.1398" effort="50" velocity="3.1416"/>
       <dynamics damping="0.1" friction="0.1"/>
     </joint>
     <joint name="J6" type="revolute">
-      <origin xyz="0 -${l_5} 0" rpy="0 0 0"/>
+      <origin xyz="0 -0.15 0" rpy="0 0 0"/>
       <parent link="J5_link"/>
       <child link="J6_link"/>
       <axis xyz="-1 0 0"/>
-      <limit lower="${j6_l * pi / 180}" upper="${j6_u * pi / 180}" effort="50" velocity="${j6_v * pi / 180}"/>
+      <limit lower="-3.9269" upper="3.9269" effort="50" velocity="3.1416"/>
       <dynamics damping="0.1" friction="0.01"/>
     </joint>
-    <joint name="imu_joint" type="fixed">
-      <origin xyz="0 0 0" rpy="0 0 0"/>
-      <parent link="base_link"/>
-      <child link="imu_link"/>
-    </joint>
-    <!-- world coords -->
-    <link name="wbase" />
-    <joint name="base_link-wbase" type="fixed">
-      <origin xyz="0 0 ${l_base}" rpy="0 0 0"/>
-      <parent link="base_link"/>
-      <child link="wbase"/>
-    </joint>
-    <!-- flange coords -->
+    <!-- Flange coordinates -->
     <link name="flange" />
     <joint name="J6-flange" type="fixed">
-      <origin xyz="${l_6} 0 0" rpy="0 0 0" />
+      <origin xyz="0.16 0 0" rpy="0 0 0" />
       <parent link="J6_link" />
       <child link="flange" />
     </joint>
-    <!-- flange1 coords -->
-    <link name="flange1" />
-    <joint name="flange-flange1" type="fixed">
-      <origin xyz="0 0 0" rpy="0 ${pi/2} 0" />
-      <parent link="flange" />
-      <child link="flange1" />
-    </joint>
-    <!-- tcp coords -->
-    <link name="tcp" />
-    <joint name="flange1-tcp" type="fixed">
-      <origin xyz="0 0 0" rpy="0 0 0" />
-      <parent link="flange1" />
-      <child link="tcp" />
-    </joint>
-    <!-- tcp right coord -->
-    <link name="tcp_right" />
-    <joint name="tcp-tcp_right" type="fixed">
-      <origin xyz="0 0.012 0.013" rpy="0 0 0" />
-      <parent link="tcp" />
-      <child link="tcp_right" />
-    </joint>
-    <!-- tcp left coord -->
-    <link name="tcp_left" />
-    <joint name="tcp-tcp_left" type="fixed">
-      <origin xyz="0 -0.012 0.013" rpy="0 0 0" />
-      <parent link="tcp" />
-      <child link="tcp_left" />
-    </joint>
-    <!-- Sensor links (not visualised) -->
-    <link name="imu_link"/>
     <!-- Add soft gripper to end of arm -->
     <xacro:include filename="$(find robot_description)/urdf/softgripper.urdf.xacro"/>
