Commit message: working Gazebo controllers

File: robot_description/urdf/robot.urdf.xacro (robot description, xacro)
@@ -1,5 +1,5 @@
 <?xml version="1.0"?>
 <robot xmlns:xacro="http://wiki.ros.org/xacro">
-  <xacro:macro name="crx10ia_l">
+  <xacro:macro name="crx_robot" params="parent">
     <material name="FANUC_Black">
       <color rgba="0 0 0 1.0"/>
@@ -45,146 +45,59 @@
     <xacro:property name="mx_2" value="0.700"/>
     <xacro:property name="my_1" value="-0.150"/>
+    <!-- world coords -->
+    <link name="wbase" />
+    <joint name="base_link-wbase" type="fixed">
+      <origin xyz="0 0 ${l_base}" rpy="0 0 0"/>
+      <parent link="base_link"/>
+      <child link="wbase"/>
+    </joint>
     <!-- links -->
     <link name="base_link">
       <visual>
-	<origin xyz="0 0 0" rpy="0 0 0"/>
-	<geometry>
-	  <mesh filename="file://$(find robot_description)/meshes/crx10ia_l/visual/base.stl" scale="0.001 0.001 0.001"/>
-	</geometry>
-	<material name="FANUC_Black"/>
-      </visual>
-      <collision>
-	<origin xyz="0 0 0" rpy="0 0 0"/>
-	<geometry>
-	  <mesh filename="file://$(find robot_description)/meshes/crx10ia_l/collision/base.stl" scale="0.001 0.001 0.001"/>
-	</geometry>
-      </collision>
-      	<inertial>
-	  <origin xyz="0 0 0" rpy="1.5708 0 0" />
-	  <mass value="10.0"/>
-	  <inertia ixx="0.02125" ixy="0" ixz="0" iyy="0.02125" iyz="0" izz="0.0125"/>
-	</inertial>
-    </link>
+        <origin xyz="0 0 0" rpy="0 0 0"/>
+        <geometry>
+          <mesh filename="file://$(find robot_description)/meshes/crx10ia_l/visual/base.stl" scale="0.001 0.001 0.001"/>
+        </geometry>
+        <material name="FANUC_Black"/>
+            </visual>
+      <collision>
+        <origin xyz="0 0 0" rpy="0 0 0"/>
+        <geometry>
+          <mesh filename="file://$(find robot_description)/meshes/crx10ia_l/collision/base.stl" scale="0.001 0.001 0.001"/>
+        </geometry>
+      </collision>
+      <inertial>
+        <origin xyz="0 0 0" rpy="1.5708 0 0" />
+        <mass value="10.0"/>
+        <inertia ixx="0.02125" ixy="0" ixz="0" iyy="0.02125" iyz="0" izz="0.0125"/>
+      </inertial>
+    </link>
+    <!-- Link to world -->
+    <joint name="base_joint" type="fixed">
+      <origin xyz="0 0 0" rpy="0 0 0"/>
+      <parent link="${parent}"/>
+      <child link="base_link" />
+    </joint>
+    <!-- J1 link and joint -->
     <link name="J1_link">
       <visual>
         <origin xyz="0 0 ${mz_1 - l_base}" rpy="0 0 0"/>
-	<geometry>
-	  <mesh filename="file://$(find robot_description)/meshes/crx10ia_l/visual/j1.stl" scale="0.001 0.001 0.001"/>
-	</geometry>
-	<material name="FANUC_White"/>
-      </visual>
+        <geometry>
+          <mesh filename="file://$(find robot_description)/meshes/crx10ia_l/visual/j1.stl" scale="0.001 0.001 0.001"/>
+        </geometry>
+        <material name="FANUC_White"/>
+            </visual>
       <collision>
         <origin xyz="0 0 ${mz_1 - l_base}" rpy="0 0 0"/>
-	<geometry>
-	  <mesh filename="file://$(find robot_description)/meshes/crx10ia_l/collision/j1.stl" scale="0.001 0.001 0.001"/>
-	</geometry>
-      </collision>
-	<inertial>
-	  <origin xyz="0 0 0" rpy="1.5708 0 0" />
-	  <mass value="5.5"/>
-	  <inertia ixx="0.03069" ixy="0" ixz="0" iyy="0.03069" iyz="0" izz="0.0176"/>
-	</inertial>
-    </link>
-    <link name="J2_link">
-      <visual>
-        <origin xyz="-${l_1} 0 ${mz_2 - l_base}" rpy="0 0 0"/>
-	<geometry>
-	  <mesh filename="file://$(find robot_description)/meshes/crx10ia_l/visual/j2.stl" scale="0.001 0.001 0.001"/>
-	</geometry>
-	<material name="FANUC_White"/>
-      </visual>
-      <collision>
-        <origin xyz="-${l_1} 0 ${mz_2 - l_base}" rpy="0 0 0"/>
-	<geometry>
-	  <mesh filename="file://$(find robot_description)/meshes/crx10ia_l/collision/j2.stl" scale="0.001 0.001 0.001"/>
-	</geometry>
-      </collision>
-	<inertial>
-	  <origin xyz="0 0 0" rpy="1.5708 0 0" />
-	  <mass value="12.1"/>
-	  <inertia ixx="0.06448" ixy="0" ixz="0" iyy="0.06448" iyz="0" izz="0.029645"/>
-	</inertial>
-    </link>
-    <link name="J3_link">
-      <visual>
-	<origin xyz="-${l_1} 0 ${mz_3 - l_base - l_2}" rpy="0 0 0"/>
-	<geometry>
-	  <mesh filename="file://$(find robot_description)/meshes/crx10ia_l/visual/j3.stl" scale="0.001 0.001 0.001"/>
-	</geometry>
-	<material name="FANUC_White"/>
-      </visual>
-      <collision>
-	<origin xyz="-${l_1} 0 ${mz_3 - l_base - l_2}" rpy="0 0 0"/>
-	<geometry>
-	  <mesh filename="file://$(find robot_description)/meshes/crx10ia_l/collision/j3.stl" scale="0.001 0.001 0.001"/>
-	</geometry>
-      </collision>
-	<inertial>
-	  <origin xyz="0 0 0" rpy="1.5708 0 0" />
-	  <mass value="2.8"/>
-	  <inertia ixx="0.00392" ixy="0" ixz="0" iyy="0.00392" iyz="0" izz="0.00252"/>
-	</inertial>
-    </link>
-    <link name="J4_link">
-      <visual>
-	<origin xyz="${mx_1 - l_1} 0 ${mz_3 - l_base - l_2 - l_3}" rpy="0 0 0"/>
-	<geometry>
-	  <mesh filename="file://$(find robot_description)/meshes/crx10ia_l/visual/j4.stl" scale="0.001 0.001 0.001"/>
-	</geometry>
-	<material name="FANUC_White"/>
-      </visual>
-      <collision>
-	<origin xyz="${mx_1 - l_1} 0 ${mz_3 - l_base - l_2 - l_3}" rpy="0 0 0"/>
-	<geometry>
-	  <mesh filename="file://$(find robot_description)/meshes/crx10ia_l/collision/j4.stl" scale="0.001 0.001 0.001"/>
-	</geometry>
-      </collision>
-	<inertial>
-	  <origin xyz="0 0 0" rpy="1.5708 0 0" />
-	  <mass value="3.4"/>
-	  <inertia ixx="0.00708" ixy="0" ixz="0" iyy="0.00708" iyz="0" izz="0.00425"/>
-	</inertial>
-    </link>
-    <link name="J5_link">
-      <visual>
-	<origin xyz="${mx_1 -l_1 - l_4} ${my_1} ${mz_3 - l_base - l_2 - l_3}" rpy="0 0 0"/>
-	<geometry>
-	  <mesh filename="file://$(find robot_description)/meshes/crx10ia_l/visual/j5.stl" scale="0.001 0.001 0.001"/>
-	</geometry>
-	<material name="FANUC_White"/>
-      </visual>
-      <collision>
-	<origin xyz="${mx_1 -l_1 - l_4} ${my_1} ${mz_3 - l_base - l_2 - l_3}" rpy="0 0 0"/>
-	<geometry>
-	  <mesh filename="file://$(find robot_description)/meshes/crx10ia_l/collision/j5.stl" scale="0.001 0.001 0.001"/>
-	</geometry>
-      </collision>
-	<inertial>
-	  <origin xyz="0 0 0" rpy="1.5708 0 0" />
-	  <mass value="1.5"/>
-	  <inertia ixx="0.00175" ixy="0" ixz="0" iyy="0.00175" iyz="0" izz="0.001"/>
-	</inertial>
-    </link>
-    <link name="J6_link">
-      <visual>
-	<origin xyz="${mx_2 -l_1 - l_4} ${my_1 + l_5} ${mz_3 - l_base - l_2 - l_3}" rpy="0 0 0"/>
-	<geometry>
-	  <mesh filename="file://$(find robot_description)/meshes/crx10ia_l/visual/j6.stl" scale="0.001 0.001 0.001"/>
-	</geometry>
-	<material name="FANUC_Black"/>
-      </visual>
-      <collision>
-	<origin xyz="${mx_2 -l_1 - l_4} ${my_1 + l_5} ${mz_3 - l_base - l_2 - l_3}" rpy="0 0 0"/>
-	<geometry>
-	  <mesh filename="file://$(find robot_description)/meshes/crx10ia_l/collision/j6.stl" scale="0.001 0.001 0.001"/>
-	</geometry>
-      </collision>
-	<inertial>
-	  <origin xyz="0 0 0" rpy="1.5708 0 0" />
-	  <mass value="0.5"/>
-	  <inertia ixx="0.00029" ixy="0" ixz="0" iyy="0.00029" iyz="0" izz="0.0004"/>
-	</inertial>
-    </link>
-    <!-- joints -->
+        <geometry>
+          <mesh filename="file://$(find robot_description)/meshes/crx10ia_l/collision/j1.stl" scale="0.001 0.001 0.001"/>
+        </geometry>
+      </collision>
+      <inertial>
+        <origin xyz="0 0 0" rpy="1.5708 0 0" />
+        <mass value="5.5"/>
+        <inertia ixx="0.03069" ixy="0" ixz="0" iyy="0.03069" iyz="0" izz="0.0176"/>
+      </inertial>
+    </link>
     <joint name="J1" type="revolute">
       <origin xyz="0 0 ${l_base}" rpy="0 0 0"/>
@@ -195,4 +108,25 @@
       <dynamics damping="0.1" friction="0.3"/>
     </joint>
+    <!-- J2 link and joint -->
+    <link name="J2_link">
+      <visual>
+        <origin xyz="-${l_1} 0 ${mz_2 - l_base}" rpy="0 0 0"/>
+        <geometry>
+          <mesh filename="file://$(find robot_description)/meshes/crx10ia_l/visual/j2.stl" scale="0.001 0.001 0.001"/>
+        </geometry>
+        <material name="FANUC_White"/>
+      </visual>
+      <collision>
+        <origin xyz="-${l_1} 0 ${mz_2 - l_base}" rpy="0 0 0"/>
+        <geometry>
+          <mesh filename="file://$(find robot_description)/meshes/crx10ia_l/collision/j2.stl" scale="0.001 0.001 0.001"/>
+        </geometry>
+      </collision>
+      <inertial>
+        <origin xyz="0 0 0" rpy="1.5708 0 0" />
+        <mass value="12.1"/>
+        <inertia ixx="0.06448" ixy="0" ixz="0" iyy="0.06448" iyz="0" izz="0.029645"/>
+      </inertial>
+    </link>
     <joint name="J2" type="revolute">
       <origin xyz="${l_1} 0 0" rpy="0 0 0"/>
@@ -203,4 +137,25 @@
       <dynamics damping="0.1" friction="0.2"/>
     </joint>
+    <!-- J3 link and joint -->
+    <link name="J3_link">
+      <visual>
+        <origin xyz="-${l_1} 0 ${mz_3 - l_base - l_2}" rpy="0 0 0"/>
+        <geometry>
+          <mesh filename="file://$(find robot_description)/meshes/crx10ia_l/visual/j3.stl" scale="0.001 0.001 0.001"/>
+        </geometry>
+        <material name="FANUC_White"/>
+      </visual>
+      <collision>
+        <origin xyz="-${l_1} 0 ${mz_3 - l_base - l_2}" rpy="0 0 0"/>
+        <geometry>
+          <mesh filename="file://$(find robot_description)/meshes/crx10ia_l/collision/j3.stl" scale="0.001 0.001 0.001"/>
+        </geometry>
+      </collision>
+      <inertial>
+        <origin xyz="0 0 0" rpy="1.5708 0 0" />
+        <mass value="2.8"/>
+        <inertia ixx="0.00392" ixy="0" ixz="0" iyy="0.00392" iyz="0" izz="0.00252"/>
+      </inertial>
+    </link>
     <joint name="J3" type="revolute">
       <origin xyz="0 0 ${l_2}" rpy="0 0 0"/>
@@ -210,4 +165,25 @@
       <limit lower="${j3_l * pi / 180}" upper="${j3_u * pi / 180}" effort="0" velocity="${j3_v * pi / 180}"/>
     </joint>
+    <!-- J4 link and joint -->
+    <link name="J4_link">
+      <visual>
+        <origin xyz="${mx_1 - l_1} 0 ${mz_3 - l_base - l_2 - l_3}" rpy="0 0 0"/>
+        <geometry>
+          <mesh filename="file://$(find robot_description)/meshes/crx10ia_l/visual/j4.stl" scale="0.001 0.001 0.001"/>
+        </geometry>
+        <material name="FANUC_White"/>
+      </visual>
+      <collision>
+        <origin xyz="${mx_1 - l_1} 0 ${mz_3 - l_base - l_2 - l_3}" rpy="0 0 0"/>
+        <geometry>
+          <mesh filename="file://$(find robot_description)/meshes/crx10ia_l/collision/j4.stl" scale="0.001 0.001 0.001"/>
+        </geometry>
+      </collision>
+      <inertial>
+        <origin xyz="0 0 0" rpy="1.5708 0 0" />
+        <mass value="3.4"/>
+        <inertia ixx="0.00708" ixy="0" ixz="0" iyy="0.00708" iyz="0" izz="0.00425"/>
+      </inertial>
+    </link>
     <joint name="J4" type="revolute">
       <origin xyz="0 0 ${l_3}" rpy="0 0 0"/>
@@ -217,4 +193,25 @@
       <limit lower="${j4_l * pi / 180}" upper="${j4_u * pi / 180}" effort="0" velocity="${j4_v * pi / 180}"/>
     </joint>
+    <!-- J5 link and joint -->
+    <link name="J5_link">
+      <visual>
+        <origin xyz="${mx_1 -l_1 - l_4} ${my_1} ${mz_3 - l_base - l_2 - l_3}" rpy="0 0 0"/>
+        <geometry>
+          <mesh filename="file://$(find robot_description)/meshes/crx10ia_l/visual/j5.stl" scale="0.001 0.001 0.001"/>
+        </geometry>
+        <material name="FANUC_White"/>
+      </visual>
+      <collision>
+        <origin xyz="${mx_1 -l_1 - l_4} ${my_1} ${mz_3 - l_base - l_2 - l_3}" rpy="0 0 0"/>
+        <geometry>
+          <mesh filename="file://$(find robot_description)/meshes/crx10ia_l/collision/j5.stl" scale="0.001 0.001 0.001"/>
+        </geometry>
+      </collision>
+      <inertial>
+        <origin xyz="0 0 0" rpy="1.5708 0 0" />
+        <mass value="1.5"/>
+        <inertia ixx="0.00175" ixy="0" ixz="0" iyy="0.00175" iyz="0" izz="0.001"/>
+      </inertial>
+    </link>
     <joint name="J5" type="revolute">
       <origin xyz="${l_4} 0 0" rpy="0 0 0"/>
@@ -224,4 +221,25 @@
       <limit lower="${j5_l * pi / 180}" upper="${j5_u * pi / 180}" effort="0" velocity="${j5_v * pi / 180}"/>
     </joint>
+    <!-- J6 link and joint -->
+    <link name="J6_link">
+      <visual>
+        <origin xyz="${mx_2 -l_1 - l_4} ${my_1 + l_5} ${mz_3 - l_base - l_2 - l_3}" rpy="0 0 0"/>
+        <geometry>
+          <mesh filename="file://$(find robot_description)/meshes/crx10ia_l/visual/j6.stl" scale="0.001 0.001 0.001"/>
+        </geometry>
+	      <material name="FANUC_Black"/>
+      </visual>
+      <collision>
+        <origin xyz="${mx_2 -l_1 - l_4} ${my_1 + l_5} ${mz_3 - l_base - l_2 - l_3}" rpy="0 0 0"/>
+        <geometry>
+          <mesh filename="file://$(find robot_description)/meshes/crx10ia_l/collision/j6.stl" scale="0.001 0.001 0.001"/>
+        </geometry>
+      </collision>
+      <inertial>
+        <origin xyz="0 0 0" rpy="1.5708 0 0" />
+        <mass value="0.5"/>
+        <inertia ixx="0.00029" ixy="0" ixz="0" iyy="0.00029" iyz="0" izz="0.0004"/>
+      </inertial>
+    </link>
     <joint name="J6" type="revolute">
       <origin xyz="0 -${l_5} 0" rpy="0 0 0"/>
@@ -231,12 +249,5 @@
       <limit lower="${j6_l * pi / 180}" upper="${j6_u * pi / 180}" effort="0" velocity="${j6_v * pi / 180}"/>
     </joint>
-    <!-- world coords -->
-    <link name="wbase" />
-    <joint name="base_link-wbase" type="fixed">
-      <origin xyz="0 0 ${l_base}" rpy="0 0 0"/>
-      <parent link="base_link"/>
-      <child link="wbase"/>
-    </joint>
-    <!-- flange coords -->
+    <!-- flange link and joint -->
     <link name="flange" />
     <joint name="J6-flange" type="fixed">

File: robot_description/urdf/robot.xacro (robot description, xacro)
@@ -1,14 +1,9 @@
 <?xml version="1.0"?>
 <robot name="crx10ia_l" xmlns:xacro="http://wiki.ros.org/xacro">
-  <!-- Arguments
-  <xacro:arg name="moveit_only" default="false"/>
-  <xacro:arg name="gazebo_classic" default="true"/> -->
   <!-- Utils -->
   <!-- <xacro:include filename="$(find robot_description)/urdf/utils.xacro" /> -->
   <!-- Robot model-->
   <xacro:include filename="$(find robot_description)/urdf/robot.urdf.xacro"/>
-  <!-- Simulation interface -->
-  <!-- <xacro:include filename="$(find robot_description)/urdf/simulation_interface.xacro"/>
-  <xacro:ros2_control name="GazeboSystem" initial_positions_file="$(find robot_moveit_config)/config/initial_positions.yaml" moveit_only="$(arg moveit_only)" gazebo_classic="$(arg gazebo_classic)"/> -->
-  <xacro:crx10ia_l/>
+  <link name="world" />
+  <xacro:crx_robot parent="world"/>
 </robot>

File: robot_moveit_config/config/crx10ia_l.urdf.xacro (robot description, xacro)
@@ -3,5 +3,5 @@
     <xacro:arg name="initial_positions_file" default="initial_positions.yaml" />
     <!-- Import crx10ia_l urdf file -->
-    <xacro:include filename="$(find robot_description)/urdf/robot.xacro" />
+    <xacro:include filename="$(find robot_description)/urdf/robot.xacro"/>
     <!-- Import control_xacro -->
     <xacro:include filename="crx10ia_l.ros2_control.xacro" />

Commit message: reintroduced utils.xacro

File: robot_description/urdf/robot.urdf.xacro (robot description, xacro)
@@ -2,16 +2,4 @@
 <robot xmlns:xacro="http://wiki.ros.org/xacro">
   <xacro:macro name="crx_robot" params="parent">
-    <material name="FANUC_Black">
-      <color rgba="0 0 0 1.0"/>
-    </material>
-    <material name="FANUC_Yellow">
-      <color rgba="1.00 0.84 0.01 1.00"/>
-    </material>
-    <material name="FANUC_Green">
-      <color rgba="0.43 0.68 0.26 1.00"/>
-    </material>
-    <material name="FANUC_White">
-      <color rgba="0.84 0.84 0.82 1.00"/>
-    </material>
     <xacro:property name="l_base" value="0.245"/>
     <xacro:property name="l_1" value="0.0"/>
@@ -67,9 +55,5 @@
         </geometry>
       </collision>
-      <inertial>
-        <origin xyz="0 0 0" rpy="1.5708 0 0" />
-        <mass value="10.0"/>
-        <inertia ixx="0.02125" ixy="0" ixz="0" iyy="0.02125" iyz="0" izz="0.0125"/>
-      </inertial>
+      <xacro:cylinder_inertia m="10.0" r="0.05" h="0.1" />
     </link>
     <!-- Link to world -->
@@ -94,9 +78,5 @@
         </geometry>
       </collision>
-      <inertial>
-        <origin xyz="0 0 0" rpy="1.5708 0 0" />
-        <mass value="5.5"/>
-        <inertia ixx="0.03069" ixy="0" ixz="0" iyy="0.03069" iyz="0" izz="0.0176"/>
-      </inertial>
+      <xacro:cylinder_inertia m="5.5" r="0.08" h="0.24" />
     </link>
     <joint name="J1" type="revolute">
@@ -123,9 +103,5 @@
         </geometry>
       </collision>
-      <inertial>
-        <origin xyz="0 0 0" rpy="1.5708 0 0" />
-        <mass value="12.1"/>
-        <inertia ixx="0.06448" ixy="0" ixz="0" iyy="0.06448" iyz="0" izz="0.029645"/>
-      </inertial>
+     <xacro:cylinder_inertia m="12.1" r="0.07" h="0.85" />
     </link>
     <joint name="J2" type="revolute">
@@ -152,9 +128,5 @@
         </geometry>
       </collision>
-      <inertial>
-        <origin xyz="0 0 0" rpy="1.5708 0 0" />
-        <mass value="2.8"/>
-        <inertia ixx="0.00392" ixy="0" ixz="0" iyy="0.00392" iyz="0" izz="0.00252"/>
-      </inertial>
+      <xacro:cylinder_inertia m="2.8" r="0.06" h="0.23" />
     </link>
     <joint name="J3" type="revolute">
@@ -180,9 +152,5 @@
         </geometry>
       </collision>
-      <inertial>
-        <origin xyz="0 0 0" rpy="1.5708 0 0" />
-        <mass value="3.4"/>
-        <inertia ixx="0.00708" ixy="0" ixz="0" iyy="0.00708" iyz="0" izz="0.00425"/>
-      </inertial>
+      <xacro:cylinder_inertia m="3.4" r="0.05" h="0.42" />
     </link>
     <joint name="J4" type="revolute">
@@ -208,9 +176,5 @@
         </geometry>
       </collision>
-      <inertial>
-        <origin xyz="0 0 0" rpy="1.5708 0 0" />
-        <mass value="1.5"/>
-        <inertia ixx="0.00175" ixy="0" ixz="0" iyy="0.00175" iyz="0" izz="0.001"/>
-      </inertial>
+      <xacro:cylinder_inertia m="1.5" r="0.05" h="0.16" />
     </link>
     <joint name="J5" type="revolute">
@@ -236,9 +200,5 @@
         </geometry>
       </collision>
-      <inertial>
-        <origin xyz="0 0 0" rpy="1.5708 0 0" />
-        <mass value="0.5"/>
-        <inertia ixx="0.00029" ixy="0" ixz="0" iyy="0.00029" iyz="0" izz="0.0004"/>
-      </inertial>
+      <xacro:cylinder_inertia m="0.5" r="0.04" h="0.06" />
     </link>
     <joint name="J6" type="revolute">

File: robot_description/urdf/robot.xacro (robot description, xacro)
@@ -2,5 +2,5 @@
 <robot name="crx10ia_l" xmlns:xacro="http://wiki.ros.org/xacro">
     <!-- Utils -->
-    <!-- <xacro:include filename="$(find robot_description)/urdf/utils.xacro" /> -->
+    <xacro:include filename="$(find robot_description)/urdf/utils.xacro" />
     <!-- Robot model-->
     <xacro:include filename="$(find robot_description)/urdf/robot.urdf.xacro"/>
