Commit message: working moveit+gazebo control

File: robot_description/urdf/robot.urdf.xacro (robot description, xacro)
@@ -1,4 +1,4 @@
 <?xml version="1.0"?>
-<robot xmlns:xacro="http://wiki.ros.org/xacro">
+<robot xmlns:xacro="http://wiki.ros.org/xacro" xmlns="http://www.w3.org/2001/XMLSchema-instance">
   <xacro:macro name="crx_robot" params="parent">
     <xacro:property name="l_base" value="0.245"/>
@@ -33,12 +33,5 @@
     <xacro:property name="mx_2" value="0.700"/>
     <xacro:property name="my_1" value="-0.150"/>
-    <!-- world coords -->
-    <link name="wbase" />
-    <joint name="base_link-wbase" type="fixed">
-      <origin xyz="0 0 ${l_base}" rpy="0 0 0"/>
-      <parent link="base_link"/>
-      <child link="wbase"/>
-    </joint>
-    <!-- links -->
+    <!-- Links -->
     <link name="base_link">
       <visual>
@@ -48,5 +41,5 @@
         </geometry>
         <material name="FANUC_Black"/>
-            </visual>
+      </visual>
       <collision>
         <origin xyz="0 0 0" rpy="0 0 0"/>
@@ -85,5 +78,5 @@
       <child link="J1_link"/>
       <axis xyz="0 0 1"/>
-      <limit lower="${j1_l * pi / 180}" upper="${j1_u * pi / 180}" effort="0" velocity="${j1_v * pi / 180}"/>
+      <limit lower="${j1_l * pi / 180}" upper="${j1_u * pi / 180}" effort="1000" velocity="${j1_v * pi / 180}"/>
       <dynamics damping="0.1" friction="0.3"/>
     </joint>
@@ -110,5 +103,5 @@
       <child link="J2_link"/>
       <axis xyz="0 1 0"/>
-      <limit lower="${j2_l * pi / 180}" upper="${j2_u * pi / 180}" effort="0" velocity="${j2_v * pi / 180}"/>
+      <limit lower="${j2_l * pi / 180}" upper="${j2_u * pi / 180}" effort="1000" velocity="${j2_v * pi / 180}"/>
       <dynamics damping="0.1" friction="0.2"/>
     </joint>
@@ -135,5 +128,6 @@
       <child link="J3_link"/>
       <axis xyz="0 -1 0"/>
-      <limit lower="${j3_l * pi / 180}" upper="${j3_u * pi / 180}" effort="0" velocity="${j3_v * pi / 180}"/>
+      <limit lower="${j3_l * pi / 180}" upper="${j3_u * pi / 180}" effort="1000" velocity="${j3_v * pi / 180}"/>
+      <dynamics damping="0.1" friction="0.2"/>
     </joint>
     <!-- J4 link and joint -->
@@ -159,5 +153,6 @@
       <child link="J4_link"/>
       <axis xyz="-1 0 0"/>
-      <limit lower="${j4_l * pi / 180}" upper="${j4_u * pi / 180}" effort="0" velocity="${j4_v * pi / 180}"/>
+      <limit lower="${j4_l * pi / 180}" upper="${j4_u * pi / 180}" effort="1000" velocity="${j4_v * pi / 180}"/>
+      <dynamics damping="0.1" friction="0.1"/>
     </joint>
     <!-- J5 link and joint -->
@@ -183,5 +178,6 @@
       <child link="J5_link"/>
       <axis xyz="0 -1 0"/>
-      <limit lower="${j5_l * pi / 180}" upper="${j5_u * pi / 180}" effort="0" velocity="${j5_v * pi / 180}"/>
+      <limit lower="${j5_l * pi / 180}" upper="${j5_u * pi / 180}" effort="1000" velocity="${j5_v * pi / 180}"/>
+      <dynamics damping="0.1" friction="0.1"/>
     </joint>
     <!-- J6 link and joint -->
@@ -207,13 +203,16 @@
       <child link="J6_link"/>
       <axis xyz="-1 0 0"/>
-      <limit lower="${j6_l * pi / 180}" upper="${j6_u * pi / 180}" effort="0" velocity="${j6_v * pi / 180}"/>
-    </joint>
-    <!-- flange link and joint -->
+      <limit lower="${j6_l * pi / 180}" upper="${j6_u * pi / 180}" effort="1000" velocity="${j6_v * pi / 180}"/>
+      <dynamics damping="0.1" friction="0.01"/>
+    </joint>
+    <!-- Flange link and joint -->
     <link name="flange" />
     <joint name="J6-flange" type="fixed">
-      <origin xyz="${l_6} 0 0" rpy="0 0 0" />
+      <origin xyz="0.16 0 0" rpy="0 0 0" />
       <parent link="J6_link" />
       <child link="flange" />
     </joint>
+    <!-- Add soft gripper to end of arm -->
+    <!-- <xacro:include filename="$(find softgripper_description)/urdf/softgripper.urdf.xacro"/> -->
   </xacro:macro>
 </robot>

File: robot_description/urdf/robot.xacro (robot description, xacro)
@@ -1,9 +1,14 @@
 <?xml version="1.0"?>
-<robot name="crx10ia_l" xmlns:xacro="http://wiki.ros.org/xacro">
-    <!-- Utils -->
-    <xacro:include filename="$(find robot_description)/urdf/utils.xacro" />
-    <!-- Robot model-->
-    <xacro:include filename="$(find robot_description)/urdf/robot.urdf.xacro"/>
-    <link name="world" />
-    <xacro:crx_robot parent="world"/>
+<robot name="crx10ial" xmlns:xacro="http://wiki.ros.org/xacro">
+  <!-- Arguments -->
+  <xacro:arg name="moveit_only" default="false"/>
+  <!-- Utils -->
+  <xacro:include filename="$(find robot_description)/urdf/utils.xacro" />
+  <!-- Robot model-->
+  <xacro:include filename="$(find robot_description)/urdf/robot.urdf.xacro"/>
+  <link name="world" />
+  <xacro:crx_robot parent="world"/>
+  <!-- Simulation interface -->
+  <xacro:include filename="$(find robot_description)/urdf/simulation_interface.xacro"/>
+  <xacro:ros2_control initial_positions_file="$(find robot_moveit_config)/config/initial_positions.yaml" moveit_only="$(arg moveit_only)"/>
 </robot>

Commit message: added cobot table URDF

File: robot_description/urdf/robot.urdf.xacro (robot description, xacro)
@@ -64,5 +64,5 @@
         </geometry>
         <material name="FANUC_White"/>
-            </visual>
+      </visual>
       <collision>
         <origin xyz="0 0 ${mz_1 - l_base}" rpy="0 0 0"/>
