Commit message: put cobot on table

File: robot_description/urdf/educational_cell.urdf.xacro (robot description, xacro)
@@ -34,4 +34,10 @@
         </inertial>
     </link>
+    <link name="world"/>
+    <joint name="table_base_joint" type="fixed">
+        <origin xyz="0 0 0" rpy="0 0 0"/>
+        <parent link="world"/>
+        <child link="table" />
+      </joint>
     <!-- Reusable wheel+bracket macro -->
     <xacro:macro name="wheel" params="prefix x y">

File: robot_description/urdf/educational_cell.xacro (robot description, xacro)
@@ -3,5 +3,5 @@
   <!-- Utils -->
   <xacro:include filename="$(find robot_description)/urdf/utils.xacro" />
-  <!-- Robot model-->
+  <!-- Table model-->
   <xacro:include filename="$(find robot_description)/urdf/educational_cell.urdf.xacro"/>
 </robot>

File: robot_description/urdf/robot.urdf.xacro (robot description, xacro)
@@ -50,7 +50,7 @@
       <xacro:cylinder_inertia m="10.0" r="0.05" h="0.1" />
     </link>
-    <!-- Link to world -->
+    <!-- Link to table -->
     <joint name="base_joint" type="fixed">
-      <origin xyz="0 0 0" rpy="0 0 0"/>
+      <origin xyz="-0.343 0 0.79" rpy="0 0 0"/>
       <parent link="${parent}"/>
       <child link="base_link" />

File: robot_description/urdf/robot.xacro (robot description, xacro)
@@ -5,8 +5,9 @@
   <!-- Utils -->
   <xacro:include filename="$(find robot_description)/urdf/utils.xacro" />
+  <!-- Table model-->
+  <xacro:include filename="$(find robot_description)/urdf/educational_cell.urdf.xacro"/>
   <!-- Robot model-->
   <xacro:include filename="$(find robot_description)/urdf/robot.urdf.xacro"/>
-  <link name="world" />
-  <xacro:crx_robot parent="world"/>
+  <xacro:crx_robot parent="table"/>
   <!-- Simulation interface -->
   <xacro:include filename="$(find robot_description)/urdf/simulation_interface.xacro"/>
